File: hw/kicad/v4.0/cmd.sch (KiCad schematic (older format))
At the start: 32 parts, among them J3 RJ45_LED, P15 CONN_01X02, U10 SN65176B, U11 SN65176B, U8 SN65176B, U9 SN65176B

Commit message: Added LCSC # to parts in 4.3 PCB
Parts:
- C112, C17, C53, C54, C55, C56: LCSC (none) -> C14663
- L7: LCSC (none) -> C85827
- R101, R102, R103, R104, R63, R66, R69, R72: LCSC (none) -> C21190
- R17, R18: LCSC (none) -> C23179
- R31: LCSC (none) -> C22765
- R62, R64, R65, R67, R68, R70, R71, R73: LCSC (none) -> C25804
- U10, U11, U8, U9: LCSC (none) -> C31302
Changed lines of the file:
@@
 EESchema Schematic File Version 4
 LIBS:stmbl_4.0-cache
-EELAYER 26 0
+EELAYER 30 0
 EELAYER END
 $Descr A4 11693 8268
@@
 F 9 "" H 0   0   50  0001 C CNN "Description"
 F 10 "Texas Instruments" H 0   0   50  0001 C CNN "Manufacturer"
+F 11 "C31302" H 5450 1400 50  0001 C CNN "LCSC"
 	1    5450 1400
 	-1   0    0    -1
@@
 F 9 "" H 0   0   50  0001 C CNN "Description"
 F 10 "" H 0   0   50  0001 C CNN "Manufacturer"
+F 11 "C21190" H 4900 1400 50  0001 C CNN "LCSC"
 	1    4900 1400
 	1    0    0    -1
@@
 F 9 "" H 0   0   50  0001 C CNN "Description"
 F 10 "" H 0   0   50  0001 C CNN "Manufacturer"
+F 11 " C14663" H 6500 1400 50  0001 C CNN "LCSC"
 	1    6500 1400
 	1    0    0    -1
@@
 F 9 "" H 0   0   50  0001 C CNN "Description"
 F 10 "Texas Instruments" H 0   0   50  0001 C CNN "Manufacturer"
+F 11 "C31302" H 5450 2800 50  0001 C CNN "LCSC"
 	1    5450 2800
 	-1   0    0    -1
@@
 F 9 "" H 0   0   50  0001 C CNN "Description"
 F 10 "" H 0   0   50  0001 C CNN "Manufacturer"
+F 11 "C21190" H 4900 2800 50  0001 C CNN "LCSC"
 	1    4900 2800
 	1    0    0    -1
@@
 F 9 "" H 0   0   50  0001 C CNN "Description"
 F 10 "" H 0   0   50  0001 C CNN "Manufacturer"
+F 11 " C14663" H 6500 2800 50  0001 C CNN "LCSC"
 	1    6500 2800
 	1    0    0    -1
@@
 F 9 "" H 0   0   50  0001 C CNN "Description"
 F 10 "Texas Instruments" H 0   0   50  0001 C CNN "Manufacturer"
+F 11 "C31302" H 5450 4200 50  0001 C CNN "LCSC"
 	1    5450 4200
 	-1   0    0    -1
@@
 F 9 "" H 0   0   50  0001 C CNN "Description"
 F 10 "" H 0   0   50  0001 C CNN "Manufacturer"
+F 11 "C21190" H 4900 4200 50  0001 C CNN "LCSC"
 	1    4900 4200
 	1    0    0    -1
@@
 F 9 "" H 0   0   50  0001 C CNN "Description"
 F 10 "" H 0   0   50  0001 C CNN "Manufacturer"
+F 11 " C14663" H 6500 4200 50  0001 C CNN "LCSC"
 	1    6500 4200
 	1    0    0    -1
@@
 F 9 "" H 0   0   50  0001 C CNN "Description"
 F 10 "Texas Instruments" H 0   0   50  0001 C CNN "Manufacturer"
+F 11 "C31302" H 5450 5600 50  0001 C CNN "LCSC"
 	1    5450 5600
 	-1   0    0    -1
@@
 F 9 "" H 0   0   50  0001 C CNN "Description"
 F 10 "" H 0   0   50  0001 C CNN "Manufacturer"
+F 11 "C21190" H 4900 5600 50  0001 C CNN "LCSC"
 	1    4900 5600
 	1    0    0    -1
@@
 F 9 "" H 0   0   50  0001 C CNN "Description"
 F 10 "" H 0   0   50  0001 C CNN "Manufacturer"
+F 11 " C14663" H 6500 5600 50  0001 C CNN "LCSC"
 	1    6500 5600
 	1    0    0    -1
@@
 F 9 "" H 0   0   50  0001 C CNN "Description"
 F 10 "" H 0   0   50  0001 C CNN "Manufacturer"
+F 11 "C22765" H 3100 4350 50  0001 C CNN "LCSC"
 	1    3100 4350
 	1    0    0    -1
@@
 F 9 "" H 0   0   50  0001 C CNN "Description"
 F 10 "" H 0   0   50  0001 C CNN "Manufacturer"
+F 11 " C14663" H 2900 4350 50  0001 C CNN "LCSC"
 	1    2900 4350
 	1    0    0    -1
@@
 F 9 "" H 0   0   50  0001 C CNN "Description"
 F 10 "" H 0   0   50  0001 C CNN "Manufacturer"
+F 11 "C23179" H 2300 3200 50  0001 C CNN "LCSC"
 	1    2300 3200
 	0    1    1    0
@@
 F 9 "" H 0   0   50  0001 C CNN "Description"
 F 10 "" H 0   0   50  0001 C CNN "Manufacturer"
+F 11 "C23179" H 2300 3900 50  0001 C CNN "LCSC"
 	1    2300 3900
 	0    1    1    0
@@
 F 9 "" H 0   0   50  0001 C CNN "Description"
 F 10 "" H 0   0   50  0001 C CNN "Manufacturer"
+F 11 "C25804" H 4900 1000 50  0001 C CNN "LCSC"
 	1    4900 1000
 	1    0    0    -1
@@
 F 9 "" H 0   0   50  0001 C CNN "Description"
 F 10 "" H 0   0   50  0001 C CNN "Manufacturer"
+F 11 "C25804" H 4900 1800 50  0001 C CNN "LCSC"
 	1    4900 1800
 	1    0    0    -1
@@
 F 9 "" H 0   0   50  0001 C CNN "Description"
 F 10 "" H 0   0   50  0001 C CNN "Manufacturer"
+F 11 "C25804" H 4900 2400 50  0001 C CNN "LCSC"
 	1    4900 2400
 	1    0    0    -1
@@
 F 9 "" H 0   0   50  0001 C CNN "Description"
 F 10 "" H 0   0   50  0001 C CNN "Manufacturer"
+F 11 "C25804" H 4900 3200 50  0001 C CNN "LCSC"
 	1    4900 3200
 	1    0    0    -1
@@
 F 9 "" H 0   0   50  0001 C CNN "Description"
 F 10 "" H 0   0   50  0001 C CNN "Manufacturer"
+F 11 "C25804" H 4900 3800 50  0001 C CNN "LCSC"
 	1    4900 3800
 	1    0    0    -1
@@
 F 9 "" H 0   0   50  0001 C CNN "Description"
 F 10 "" H 0   0   50  0001 C CNN "Manufacturer"
+F 11 "C25804" H 4900 4600 50  0001 C CNN "LCSC"
 	1    4900 4600
 	1    0    0    -1
@@
 F 9 "" H 0   0   50  0001 C CNN "Description"
 F 10 "" H 0   0   50  0001 C CNN "Manufacturer"
+F 11 "C25804" H 4900 5200 50  0001 C CNN "LCSC"
 	1    4900 5200
 	1    0    0    -1
@@
 F 9 "" H 0   0   50  0001 C CNN "Description"
 F 10 "" H 0   0   50  0001 C CNN "Manufacturer"
+F 11 "C25804" H 4900 6000 50  0001 C CNN "LCSC"
 	1    4900 6000
 	1    0    0    -1
@@
 F 9 "" H 0   0   50  0001 C CNN "Description"
 F 10 "" H 0   0   50  0001 C CNN "Manufacturer"
+F 11 "C21190" H 6900 1600 50  0001 C CNN "LCSC"
 	1    6900 1600
 	1    0    0    -1
@@
 F 9 "" H 0   0   50  0001 C CNN "Description"
 F 10 "" H 0   0   50  0001 C CNN "InternalName"
+F 11 "C21190" H 6900 3000 50  0001 C CNN "LCSC"
 	1    6900 3000
 	1    0    0    -1
@@
 F 9 "" H 0   0   50  0001 C CNN "Description"
 F 10 "" H 0   0   50  0001 C CNN "Manufacturer"
+F 11 "C21190" H 6900 4400 50  0001 C CNN "LCSC"
 	1    6900 4400
 	1    0    0    -1
@@
 F 9 "" H 0   0   50  0001 C CNN "Description"
 F 10 "" H 0   0   50  0001 C CNN "Manufacturer"
+F 11 "C21190" H 6900 5800 50  0001 C CNN "LCSC"
 	1    6900 5800
 	1    0    0    -1
@@
 F 9 "" H 0   0   50  0001 C CNN "Description"
 F 10 "Murata" H 0   0   50  0001 C CNN "Manufacturer"
+F 11 "C85827" H 7700 950 50  0001 C CNN "LCSC"
 	1    7700 950
 	0    -1   -1   0
@@
 F 9 "" H 0   0   50  0001 C CNN "Description"
 F 10 "" H 0   0   50  0001 C CNN "Manufacturer"
+F 11 " C14663" H 8100 1200 50  0001 C CNN "LCSC"
 	1    8100 1200
 	1    0    0    -1
