File: hw/kicad/v4.0/cmd.sch (KiCad schematic (older format))
At the start: 32 parts, among them J3 RJ45_LED, P15 CONN_01X02, U10 SN65176B, U11 SN65176B, U8 SN65176B, U9 SN65176B

Commit message: WIP LCSC
Parts:
- C112, C17, C53, C54, C55, C56: LCSC (none) -> C14663
- J3: LCSC (none) -> C138392
- P15: LCSC (none) -> C441171
Changed lines of the file:
@@
 EESchema Schematic File Version 4
-LIBS:stmbl_4.0-cache
-EELAYER 26 0
+EELAYER 30 0
 EELAYER END
 $Descr A4 11693 8268
@@
 F 9 "" H 0   0   50  0001 C CNN "Description"
 F 10 "METZ CONNECT" H 0   0   50  0001 C CNN "Manufacturer"
+F 11 "C138392" H 3000 3500 50  0001 C CNN "LCSC"
 	1    3000 3500
 	0    -1   1    0
@@
 F 9 "" H 0   0   50  0001 C CNN "Description"
 F 10 "" H 0   0   50  0001 C CNN "Manufacturer"
+F 11 "C14663" H 6500 1400 50  0001 C CNN "LCSC"
 	1    6500 1400
 	1    0    0    -1
@@
 F 9 "" H 0   0   50  0001 C CNN "Description"
 F 10 "" H 0   0   50  0001 C CNN "Manufacturer"
+F 11 "C14663" H 6500 2800 50  0001 C CNN "LCSC"
 	1    6500 2800
 	1    0    0    -1
@@
 F 9 "" H 0   0   50  0001 C CNN "Description"
 F 10 "" H 0   0   50  0001 C CNN "Manufacturer"
+F 11 "C14663" H 6500 4200 50  0001 C CNN "LCSC"
 	1    6500 4200
 	1    0    0    -1
@@
 F 9 "" H 0   0   50  0001 C CNN "Description"
 F 10 "" H 0   0   50  0001 C CNN "Manufacturer"
+F 11 "C14663" H 6500 5600 50  0001 C CNN "LCSC"
 	1    6500 5600
 	1    0    0    -1
@@
 F 9 "" H 0   0   50  0001 C CNN "Description"
 F 10 "" H 0   0   50  0001 C CNN "Manufacturer"
+F 11 "C14663" H 2900 4350 50  0001 C CNN "LCSC"
 	1    2900 4350
 	1    0    0    -1
@@
 F 9 "" H 0   0   50  0001 C CNN "Description"
 F 10 "" H 0   0   50  0001 C CNN "Manufacturer"
+F 11 "C14663" H 8100 1200 50  0001 C CNN "LCSC"
 	1    8100 1200
 	1    0    0    -1
@@
 F 9 "" H 0   0   50  0001 C CNN "Description"
 F 10 "Phoenix" H 0   0   50  0001 C CNN "Manufacturer"
+F 11 "C441171" H 4400 4200 50  0001 C CNN "LCSC"
 	1    4400 4200
 	-1   0    0    -1
