File: hw/kicad/v4.0/cmd.sch (KiCad schematic (older format))
At the start: 32 parts, among them J3 RJ45_LED, P15 CONN_01X02, U10 SN65176B, U11 SN65176B, U8 SN65176B, U9 SN65176B

Commit message: Changed 120uf 1808 to 1210 100uF
Parts:
- C112, C17, C53, C54, C55, C56: LCSC C14663 -> C14663
Changed lines of the file:
@@
 F 9 "" H 0   0   50  0001 C CNN "Description"
 F 10 "" H 0   0   50  0001 C CNN "Manufacturer"
-F 11 " C14663" H 6500 1400 50  0001 C CNN "LCSC"
+F 11 "C14663" H 6500 1400 50  0001 C CNN "LCSC"
 	1    6500 1400
 	1    0    0    -1
@@
 F 9 "" H 0   0   50  0001 C CNN "Description"
 F 10 "" H 0   0   50  0001 C CNN "Manufacturer"
-F 11 " C14663" H 6500 2800 50  0001 C CNN "LCSC"
+F 11 "C14663" H 6500 2800 50  0001 C CNN "LCSC"
 	1    6500 2800
 	1    0    0    -1
@@
 F 9 "" H 0   0   50  0001 C CNN "Description"
 F 10 "" H 0   0   50  0001 C CNN "Manufacturer"
-F 11 " C14663" H 6500 4200 50  0001 C CNN "LCSC"
+F 11 "C14663" H 6500 4200 50  0001 C CNN "LCSC"
 	1    6500 4200
 	1    0    0    -1
@@
 F 9 "" H 0   0   50  0001 C CNN "Description"
 F 10 "" H 0   0   50  0001 C CNN "Manufacturer"
-F 11 " C14663" H 6500 5600 50  0001 C CNN "LCSC"
+F 11 "C14663" H 6500 5600 50  0001 C CNN "LCSC"
 	1    6500 5600
 	1    0    0    -1
@@
 F 9 "" H 0   0   50  0001 C CNN "Description"
 F 10 "" H 0   0   50  0001 C CNN "Manufacturer"
-F 11 " C14663" H 2900 4350 50  0001 C CNN "LCSC"
+F 11 "C14663" H 2900 4350 50  0001 C CNN "LCSC"
 	1    2900 4350
 	1    0    0    -1
@@
 F 9 "" H 0   0   50  0001 C CNN "Description"
 F 10 "" H 0   0   50  0001 C CNN "Manufacturer"
-F 11 " C14663" H 8100 1200 50  0001 C CNN "LCSC"
+F 11 "C14663" H 8100 1200 50  0001 C CNN "LCSC"
 	1    8100 1200
 	1    0    0    -1

Commit message: Switch some 2.2uf 0603 to 1uf bypass to get 50V version on jlcpcb
Change 2.2uf 0603 to 0805 on iram to get 50V version on jlcpcb
other cleanup
Parts:
- C112, C17, C53, C54, C55, C56: Manufacturer (none) -> YAGEO; Manufacturer No (none) -> CC0603KRX7R9BB104
- J3: LCSC C138392 -> (none)
- P15: LCSC C441171 -> (none)
Changed lines of the file:
@@
 F 9 "" H 0   0   50  0001 C CNN "Description"
 F 10 "METZ CONNECT" H 0   0   50  0001 C CNN "Manufacturer"
-F 11 "C138392" H 3000 3500 50  0001 C CNN "LCSC"
+F 11 "" H 3000 3500 50  0001 C CNN "LCSC"
 	1    3000 3500
 	0    -1   1    0
@@
 F 5 "50V" H 6525 1600 50  0001 C CNN "Voltage"
 F 6 "" H 6500 1400 60  0001 C CNN "InternalName"
-F 7 "" H 6500 1400 60  0001 C CNN "Manufacturer No"
+F 7 "CC0603KRX7R9BB104 " H 6500 1400 60  0001 C CNN "Manufacturer No"
 F 8 "" H 6500 1400 60  0001 C CNN "Source"
 F 9 "" H 0   0   50  0001 C CNN "Description"
-F 10 "" H 0   0   50  0001 C CNN "Manufacturer"
+F 10 "YAGEO" H 0   0   50  0001 C CNN "Manufacturer"
 F 11 "C14663" H 6500 1400 50  0001 C CNN "LCSC"
 	1    6500 1400
@@
 F 5 "50V" H 6500 2800 50  0001 C CNN "Voltage"
 F 6 "" H 6500 2800 60  0001 C CNN "InternalName"
-F 7 "" H 6500 2800 60  0001 C CNN "Manufacturer No"
+F 7 "CC0603KRX7R9BB104 " H 6500 2800 60  0001 C CNN "Manufacturer No"
 F 8 "" H 6500 2800 60  0001 C CNN "Source"
 F 9 "" H 0   0   50  0001 C CNN "Description"
-F 10 "" H 0   0   50  0001 C CNN "Manufacturer"
+F 10 "YAGEO" H 0   0   50  0001 C CNN "Manufacturer"
 F 11 "C14663" H 6500 2800 50  0001 C CNN "LCSC"
 	1    6500 2800
@@
 F 5 "50V" H 6525 4400 50  0001 C CNN "Voltage"
 F 6 "" H 6500 4200 60  0001 C CNN "InternalName"
-F 7 "" H 6500 4200 60  0001 C CNN "Manufacturer No"
+F 7 "CC0603KRX7R9BB104 " H 6500 4200 60  0001 C CNN "Manufacturer No"
 F 8 "" H 6500 4200 60  0001 C CNN "Source"
 F 9 "" H 0   0   50  0001 C CNN "Description"
-F 10 "" H 0   0   50  0001 C CNN "Manufacturer"
+F 10 "YAGEO" H 0   0   50  0001 C CNN "Manufacturer"
 F 11 "C14663" H 6500 4200 50  0001 C CNN "LCSC"
 	1    6500 4200
@@
 F 5 "50V" H 6525 5800 50  0001 C CNN "Voltage"
 F 6 "" H 6500 5600 60  0001 C CNN "InternalName"
-F 7 "" H 6500 5600 60  0001 C CNN "Manufacturer No"
+F 7 "CC0603KRX7R9BB104 " H 6500 5600 60  0001 C CNN "Manufacturer No"
 F 8 "" H 6500 5600 60  0001 C CNN "Source"
 F 9 "" H 0   0   50  0001 C CNN "Description"
-F 10 "" H 0   0   50  0001 C CNN "Manufacturer"
+F 10 "YAGEO" H 0   0   50  0001 C CNN "Manufacturer"
 F 11 "C14663" H 6500 5600 50  0001 C CNN "LCSC"
 	1    6500 5600
@@
 F 5 "50V" H 2925 4550 50  0001 C CNN "Voltage"
 F 6 "" H 2900 4350 60  0001 C CNN "InternalName"
-F 7 "" H 2900 4350 60  0001 C CNN "Manufacturer No"
+F 7 "CC0603KRX7R9BB104 " H 2900 4350 60  0001 C CNN "Manufacturer No"
 F 8 "" H 2900 4350 60  0001 C CNN "Source"
 F 9 "" H 0   0   50  0001 C CNN "Description"
-F 10 "" H 0   0   50  0001 C CNN "Manufacturer"
+F 10 "YAGEO" H 0   0   50  0001 C CNN "Manufacturer"
 F 11 "C14663" H 2900 4350 50  0001 C CNN "LCSC"
 	1    2900 4350
@@
 F 5 "50V" H 8125 1400 50  0001 C CNN "Voltage"
 F 6 "" H 8100 1200 60  0001 C CNN "InternalName"
-F 7 "" H 8100 1200 60  0001 C CNN "Manufacturer No"
+F 7 "CC0603KRX7R9BB104 " H 8100 1200 60  0001 C CNN "Manufacturer No"
 F 8 "" H 8100 1200 60  0001 C CNN "Source"
 F 9 "" H 0   0   50  0001 C CNN "Description"
-F 10 "" H 0   0   50  0001 C CNN "Manufacturer"
+F 10 "YAGEO" H 0   0   50  0001 C CNN "Manufacturer"
 F 11 "C14663" H 8100 1200 50  0001 C CNN "LCSC"
 	1    8100 1200
@@
 F 9 "" H 0   0   50  0001 C CNN "Description"
 F 10 "Phoenix" H 0   0   50  0001 C CNN "Manufacturer"
-F 11 "C441171" H 4400 4200 50  0001 C CNN "LCSC"
+F 11 "" H 4400 4200 50  0001 C CNN "LCSC"
 	1    4400 4200
 	-1   0    0    -1
