File: hw/kicad/v4.0/f3.sch (KiCad schematic (older format))
At the start: 34 parts, among them P11 USB_OTG, P12 CONN_01X04, P7 CONN_01X04, T1 testpoint, T2 testpoint, T44 testpoint, T45 testpoint, T46 testpoint, U21 USBLC6-4SC6, U25 STM32F303CBTx, U29 USBLC6-4SC6, Y1 8M

Commit message: Added LCSC # to parts in 4.3 PCB
Parts:
- C10, C128, C2, C7, C78, C79, C82, C83, C9: LCSC (none) -> C14663
- C141: LCSC (none) -> C23630
- C5, C6: LCSC (none) -> C1647
- D1: LCSC (none) -> C84256
- L1: LCSC (none) -> C85827
- R118, R129, R2: LCSC (none) -> C21190
- R150: LCSC (none) -> C22843
- R151, R152: LCSC (none) -> C23345
- R8: LCSC (none) -> C23179
- U21, U29: LCSC (none) -> C252436
- U25: LCSC (none) -> C108516
Changed lines of the file:
@@
 EESchema Schematic File Version 4
 LIBS:stmbl_4.0-cache
-EELAYER 26 0
+EELAYER 30 0
 EELAYER END
 $Descr User 19685 7874
@@
 F 9 "" H 0   0   50  0001 C CNN "Description"
 F 10 "" H 0   0   50  0001 C CNN "Manufacturer"
+F 11 " C14663" H 9700 950 50  0001 C CNN "LCSC"
 	1    9700 950
 	1    0    0    -1
@@
 F 9 "" H 0   0   50  0001 C CNN "Description"
 F 10 "" H 0   0   50  0001 C CNN "Manufacturer"
+F 11 " C14663" H 9800 950 50  0001 C CNN "LCSC"
 	1    9800 950
 	1    0    0    -1
@@
 F 9 "" H 0   0   50  0001 C CNN "Description"
 F 10 "" H 0   0   50  0001 C CNN "Manufacturer"
+F 11 " C14663" H 9900 950 50  0001 C CNN "LCSC"
 	1    9900 950
 	1    0    0    -1
@@
 F 9 "" H 0   0   50  0001 C CNN "Description"
 F 10 "" H 0   0   50  0001 C CNN "Manufacturer"
+F 11 " C14663" H 10000 950 50  0001 C CNN "LCSC"
 	1    10000 950
 	1    0    0    -1
@@
 F 9 "" H 0   0   50  0001 C CNN "Description"
 F 10 "" H 0   0   50  0001 C CNN "Manufacturer"
+F 11 "C1647" H 8350 2000 50  0001 C CNN "LCSC"
 	1    8350 2000
 	0    1    1    0
@@
 F 9 "" H 0   0   50  0001 C CNN "Description"
 F 10 "" H 0   0   50  0001 C CNN "Manufacturer"
+F 11 "C1647" H 8350 2300 50  0001 C CNN "LCSC"
 	1    8350 2300
 	0    1    1    0
@@
 F 9 "" H 0   0   50  0001 C CNN "Description"
 F 10 "" H 0   0   50  0001 C CNN "Manufacturer"
+F 11 " C14663" H 7800 2150 50  0001 C CNN "LCSC"
 	1    7800 2150
 	1    0    0    -1
@@
 F 9 "" H 0   0   50  0001 C CNN "Description"
 F 10 "" H 0   0   50  0001 C CNN "Manufacturer"
+F 11 " C14663" H 8850 1500 50  0001 C CNN "LCSC"
 	1    8850 1500
 	0    1    1    0
@@
 F 9 "" H 0   0   50  0001 C CNN "Description"
 F 10 "" H 0   0   50  0001 C CNN "Manufacturer"
+F 11 "C21190" H 7500 1950 50  0001 C CNN "LCSC"
 	1    7500 1950
 	1    0    0    -1
@@
 F 9 "" H 0   0   50  0001 C CNN "InternalName"
 F 10 "STMicroelectronics" H 0   0   50  0001 C CNN "Manufacturer"
+F 11 "C252436" H 9400 6600 50  0001 C CNN "LCSC"
 	1    9400 6600
 	1    0    0    -1
@@
 F 9 "" H 0   0   50  0001 C CNN "Description"
 F 10 "STMicroelectronics" H 0   0   50  0001 C CNN "Manufacturer"
+F 11 "C108516" H 9800 3000 50  0001 C CNN "LCSC"
 	1    9800 3000
 	1    0    0    -1
@@
 F 9 "" H 0   0   50  0001 C CNN "Description"
 F 10 "" H 0   0   50  0001 C CNN "Manufacturer"
+F 11 "C21190" H 10750 4400 50  0001 C CNN "LCSC"
 	1    10750 4400
 	0    1    1    0
@@
 F 9 "" H 0   0   50  0001 C CNN "Description"
 F 10 "Lite-On" H 0   0   50  0001 C CNN "Manufacturer"
+F 11 "C84256" H 10900 3600 50  0001 C CNN "LCSC"
 	1    10900 3600
 	-1   0    0    1
@@
 F 9 "" H 0   0   50  0001 C CNN "Description"
 F 10 "" H 0   0   50  0001 C CNN "Manufacturer"
+F 11 "C23179" H 11350 3600 50  0001 C CNN "LCSC"
 	1    11350 3600
 	0    1    1    0
@@
 F 9 "" H 0   0   50  0001 C CNN "Description"
 F 10 "Murata" H 0   0   50  0001 C CNN "Manufacturer"
+F 11 "C85827" H 10600 1200 50  0001 C CNN "LCSC"
 	1    10600 1200
 	0    -1   -1   0
@@
 F 9 "" H 0   0   50  0001 C CNN "Description"
 F 10 "" H 0   0   50  0001 C CNN "Manufacturer"
+F 11 " C14663" H 11000 1000 50  0001 C CNN "LCSC"
 	1    11000 1000
 	1    0    0    -1
@@
 F 9 "" H 0   0   50  0001 C CNN "Description"
 F 10 "" H 0   0   50  0001 C CNN "Manufacturer"
+F 11 " C14663" H 7450 6600 50  0001 C CNN "LCSC"
 	1    7450 6600
 	1    0    0    -1
@@
 F 9 "" H 0   0   50  0001 C CNN "InternalName"
 F 10 "STMicroelectronics" H 0   0   50  0001 C CNN "Manufacturer"
+F 11 "C252436" H 4350 5650 50  0001 C CNN "LCSC"
 	1    4350 5650
 	1    0    0    -1
@@
 F 9 "" H 0   0   50  0001 C CNN "Description"
 F 10 "" H 0   0   50  0001 C CNN "Manufacturer"
+F 11 " C14663" H 4100 6500 50  0001 C CNN "LCSC"
 	1    4100 6500
 	1    0    0    -1
@@
 F 9 "" H 0   0   50  0001 C CNN "Description"
 F 10 "" H 0   0   50  0001 C CNN "Manufacturer"
+F 11 "C23345" H 7550 5550 50  0001 C CNN "LCSC"
 	1    7550 5550
 	0    1    1    0
@@
 F 9 "" H 0   0   50  0001 C CNN "Description"
 F 10 "" H 0   0   50  0001 C CNN "Manufacturer"
+F 11 "C23345" H 7550 5650 50  0001 C CNN "LCSC"
 	1    7550 5650
 	0    1    1    0
@@
 F 9 "" H 0   0   50  0001 C CNN "Description"
 F 10 "" H 0   0   50  0001 C CNN "Manufacturer"
+F 11 "C22843" H 7300 5300 50  0001 C CNN "LCSC"
 	1    7300 5300
 	-1   0    0    1
@@
 F 9 "" H 0   0   50  0001 C CNN "Description"
 F 10 "" H 0   0   50  0001 C CNN "Manufacturer"
+F 11 "C21190" H 8850 2300 50  0001 C CNN "LCSC"
 	1    8850 2300
 	0    1    1    0
@@
 F 9 "" H 0   0   50  0001 C CNN "Description"
 F 10 "" H 0   0   50  0001 C CNN "Manufacturer"
+F 11 "C23630" H 10200 950 50  0001 C CNN "LCSC"
 	1    10200 950
 	1    0    0    -1
