File: hw/kicad/v4.0/f3.sch (KiCad schematic (older format))
At the start: 34 parts, among them P11 USB_OTG, P12 CONN_01X04, P7 CONN_01X04, T1 testpoint, T2 testpoint, T44 testpoint, T45 testpoint, T46 testpoint, U21 USBLC6-4SC6, U25 STM32F303CBTx, U29 USBLC6-4SC6, Y1 8M

Commit message: WIP LCSC
Parts:
- C10, C128, C2, C7, C78, C79, C82, C83, C9: LCSC (none) -> C14663
- P11: LCSC (none) -> C145792
- Y1: LCSC (none) -> C389778
Changed lines of the file:
@@
 EESchema Schematic File Version 4
-LIBS:stmbl_4.0-cache
-EELAYER 26 0
+EELAYER 30 0
 EELAYER END
 $Descr User 19685 7874
@@
 F 9 "" H 0   0   50  0001 C CNN "Description"
 F 10 "" H 0   0   50  0001 C CNN "Manufacturer"
+F 11 "C14663" H 9700 950 50  0001 C CNN "LCSC"
 	1    9700 950
 	1    0    0    -1
@@
 F 9 "" H 0   0   50  0001 C CNN "Description"
 F 10 "" H 0   0   50  0001 C CNN "Manufacturer"
+F 11 "C14663" H 9800 950 50  0001 C CNN "LCSC"
 	1    9800 950
 	1    0    0    -1
@@
 F 9 "" H 0   0   50  0001 C CNN "Description"
 F 10 "" H 0   0   50  0001 C CNN "Manufacturer"
+F 11 "C14663" H 9900 950 50  0001 C CNN "LCSC"
 	1    9900 950
 	1    0    0    -1
@@
 F 9 "" H 0   0   50  0001 C CNN "Description"
 F 10 "" H 0   0   50  0001 C CNN "Manufacturer"
+F 11 "C14663" H 10000 950 50  0001 C CNN "LCSC"
 	1    10000 950
 	1    0    0    -1
@@
 F 9 "" H 0   0   50  0001 C CNN "Description"
 F 10 "Abracon LLC" H 0   0   50  0001 C CNN "Manufacturer"
+F 11 "C389778" H 8600 2150 50  0001 C CNN "LCSC"
 	1    8600 2150
 	0    1    1    0
@@
 F 9 "" H 0   0   50  0001 C CNN "Description"
 F 10 "" H 0   0   50  0001 C CNN "Manufacturer"
+F 11 "C14663" H 7800 2150 50  0001 C CNN "LCSC"
 	1    7800 2150
 	1    0    0    -1
@@
 F 9 "" H 0   0   50  0001 C CNN "Description"
 F 10 "" H 0   0   50  0001 C CNN "Manufacturer"
+F 11 "C14663" H 8850 1500 50  0001 C CNN "LCSC"
 	1    8850 1500
 	0    1    1    0
@@
 F 9 "" H 0   0   50  0001 C CNN "Description"
 F 10 "" H 0   0   50  0001 C CNN "Manufacturer"
+F 11 "C14663" H 11000 1000 50  0001 C CNN "LCSC"
 	1    11000 1000
 	1    0    0    -1
@@
 F 9 "" H 0   0   50  0001 C CNN "Description"
 F 10 "" H 0   0   50  0001 C CNN "Manufacturer"
+F 11 "C14663" H 7450 6600 50  0001 C CNN "LCSC"
 	1    7450 6600
 	1    0    0    -1
@@
 F 9 "" H 0   0   50  0001 C CNN "Description"
 F 10 "" H 0   0   50  0001 C CNN "Manufacturer"
+F 11 "C14663" H 4100 6500 50  0001 C CNN "LCSC"
 	1    4100 6500
 	1    0    0    -1
@@
 F 9 "" H 0   0   50  0001 C CNN "Description"
 F 10 "Molex" H 0   0   50  0001 C CNN "Manufacturer"
+F 11 "C145792" H 6900 5650 50  0001 C CNN "LCSC"
 	1    6900 5650
 	0    -1   1    0
