File: hw/kicad/v4.0/f4.sch (KiCad schematic (older format))
At the start: 37 parts, among them P1 USB_OTG, U1 USBLC6-4SC6, U20 USBLC6-4SC6, U22 USBLC6-4SC6, U23 USBLC6-4SC6, U26 STM32F405VG, Y2 8M

Commit message: Added LCSC # to parts in 4.3 PCB
Parts:
- C1, C119, C16, C29, C61, C66, C67, C77, C80, C84, C85, C86, C87, C89: LCSC (none) -> C14663
- C31, C32: LCSC (none) -> C1647
- C64, C81: LCSC (none) -> C1588
- C65, C88, C90: LCSC (none) -> C23630
- L3: LCSC (none) -> C85827
- R1: LCSC (none) -> C22765
- R116: LCSC (none) -> C25804
- R117, R121, R122, R153, R61: LCSC (none) -> C21190
- U1, U20, U22, U23: LCSC (none) -> C252436
- U26: LCSC (none) -> C56621
Changed lines of the file:
@@
 EESchema Schematic File Version 4
 LIBS:stmbl_4.0-cache
-EELAYER 26 0
+EELAYER 30 0
 EELAYER END
 $Descr A3 16535 11693
@@
 F 9 "" H 0   0   50  0001 C CNN "Description"
 F 10 "STMicroelectronics" H 0   0   50  0001 C CNN "Manufacturer"
+F 11 "C56621" H 10200 5500 50  0001 C CNN "LCSC"
 	1    10200 5500
 	1    0    0    -1
@@
 F 9 "" H 0   0   50  0001 C CNN "Description"
 F 10 "" H 0   0   50  0001 C CNN "Manufacturer"
+F 11 "C1647" H 4350 3400 50  0001 C CNN "LCSC"
 	1    4350 3400
 	0    1    1    0
@@
 F 9 "" H 0   0   50  0001 C CNN "Description"
 F 10 "" H 0   0   50  0001 C CNN "Manufacturer"
+F 11 "C1647" H 4350 4000 50  0001 C CNN "LCSC"
 	1    4350 4000
 	0    1    1    0
@@
 F 9 "" H 0   0   50  0001 C CNN "Description"
 F 10 "" H 0   0   50  0001 C CNN "Manufacturer"
+F 11 "C23630" H 11600 8750 50  0001 C CNN "LCSC"
 	1    11600 8750
 	1    0    0    -1
@@
 F 9 "" H 0   0   50  0001 C CNN "Description"
 F 10 "" H 0   0   50  0001 C CNN "Manufacturer"
+F 11 "C23630" H 11100 8750 50  0001 C CNN "LCSC"
 	1    11100 8750
 	1    0    0    -1
@@
 F 9 "" H 0   0   50  0001 C CNN "Description"
 F 10 "" H 0   0   50  0001 C CNN "Manufacturer"
+F 11 " C14663" H 11400 2150 50  0001 C CNN "LCSC"
 	1    11400 2150
 	1    0    0    -1
@@
 F 9 "" H 0   0   50  0001 C CNN "Description"
 F 10 "" H 0   0   50  0001 C CNN "Manufacturer"
+F 11 " C14663" H 10900 2150 50  0001 C CNN "LCSC"
 	1    10900 2150
 	1    0    0    -1
@@
 F 9 "" H 0   0   50  0001 C CNN "Description"
 F 10 "" H 0   0   50  0001 C CNN "Manufacturer"
+F 11 " C14663" H 10600 2150 50  0001 C CNN "LCSC"
 	1    10600 2150
 	1    0    0    -1
@@
 F 9 "" H 0   0   50  0001 C CNN "Description"
 F 10 "" H 0   0   50  0001 C CNN "Manufacturer"
+F 11 " C14663" H 10300 2150 50  0001 C CNN "LCSC"
 	1    10300 2150
 	1    0    0    -1
@@
 F 9 "" H 0   0   50  0001 C CNN "Description"
 F 10 "" H 0   0   50  0001 C CNN "Manufacturer"
+F 11 " C14663" H 10000 2150 50  0001 C CNN "LCSC"
 	1    10000 2150
 	1    0    0    -1
@@
 F 9 "" H 0   0   50  0001 C CNN "Description"
 F 10 "" H 0   0   50  0001 C CNN "Manufacturer"
+F 11 " C14663" H 9700 2150 50  0001 C CNN "LCSC"
 	1    9700 2150
 	1    0    0    -1
@@
 F 9 "" H 0   0   50  0001 C CNN "Description"
 F 10 "" H 0   0   50  0001 C CNN "Manufacturer"
+F 11 " C14663" H 9400 2150 50  0001 C CNN "LCSC"
 	1    9400 2150
 	1    0    0    -1
@@
 F 9 "" H 0   0   50  0001 C CNN "Description"
 F 10 "" H 0   0   50  0001 C CNN "Manufacturer"
+F 11 "C23630" H 8400 2150 50  0001 C CNN "LCSC"
 	1    8400 2150
 	1    0    0    -1
@@
 F 9 "" H 0   0   50  0001 C CNN "Description"
 F 10 "Murata" H 0   0   50  0001 C CNN "Manufacturer"
+F 11 "C85827" H 8900 2400 50  0001 C CNN "LCSC"
 	1    8900 2400
 	0    -1   -1   0
@@
 F 9 "" H 0   0   50  0001 C CNN "Description"
 F 10 "" H 0   0   50  0001 C CNN "Manufacturer"
+F 11 " C14663" H 4600 2850 50  0001 C CNN "LCSC"
 	1    4600 2850
 	1    0    0    -1
@@
 F 9 "" H 0   0   50  0001 C CNN "Voltage"
 F 10 "STMicroelectronics" H 0   0   50  0001 C CNN "Manufacturer"
+F 11 "C252436" H 2800 6550 50  0001 C CNN "LCSC"
 	1    2800 6550
 	1    0    0    -1
@@
 F 9 "" H 0   0   50  0001 C CNN "Description"
 F 10 "" H 0   0   50  0001 C CNN "Manufacturer"
+F 11 "C25804" H 7850 9050 50  0001 C CNN "LCSC"
 	1    7850 9050
 	1    0    0    -1
@@
 F 9 "" H 0   0   50  0001 C CNN "Description"
 F 10 "" H 0   0   50  0001 C CNN "Manufacturer"
+F 11 "C21190" H 7850 9550 50  0001 C CNN "LCSC"
 	1    7850 9550
 	1    0    0    -1
@@
 F 9 "" H 0   0   50  0001 C CNN "Description"
 F 10 "" H 0   0   50  0001 C CNN "Manufacturer"
+F 11 "C21190" H 8750 9050 50  0001 C CNN "LCSC"
 	1    8750 9050
 	1    0    0    -1
@@
 F 9 "" H 0   0   50  0001 C CNN "Description"
 F 10 "" H 0   0   50  0001 C CNN "Manufacturer"
+F 11 "C21190" H 8750 9550 50  0001 C CNN "LCSC"
 	1    8750 9550
 	1    0    0    -1
@@
 F 9 "" H 0   0   50  0001 C CNN "Description"
 F 10 "" H 0   0   50  0001 C CNN "Manufacturer"
+F 11 "C1588" H 8950 9550 50  0001 C CNN "LCSC"
 	1    8950 9550
 	1    0    0    -1
@@
 F 9 "" H 0   0   50  0001 C CNN "Description"
 F 10 "" H 0   0   50  0001 C CNN "Manufacturer"
+F 11 "C1588" H 8050 9550 50  0001 C CNN "LCSC"
 	1    8050 9550
 	1    0    0    -1
@@
 F 9 "" H 0   0   50  0001 C CNN "Description"
 F 10 "" H 0   0   50  0001 C CNN "Manufacturer"
+F 11 "C21190" H 4850 2750 50  0001 C CNN "LCSC"
 	1    4850 2750
 	1    0    0    -1
@@
 F 9 "" H 0   0   50  0001 C CNN "Description"
 F 10 "" H 0   0   50  0001 C CNN "Manufacturer"
+F 11 " C14663" H 2800 7050 50  0001 C CNN "LCSC"
 	1    2800 7050
 	0    1    1    0
@@
 F 9 "" H 0   0   50  0001 C CNN "Description"
 F 10 "" H 0   0   50  0001 C CNN "Manufacturer"
+F 11 " C14663" H 8100 2150 50  0001 C CNN "LCSC"
 	1    8100 2150
 	1    0    0    -1
@@
 F 9 "" H 0   0   50  0001 C CNN "Description"
 F 10 "" H 0   0   50  0001 C CNN "Manufacturer"
+F 11 " C14663" H 850 6650 50  0001 C CNN "LCSC"
 	1    850  6650
 	1    0    0    -1
@@
 F 9 "" H 0   0   50  0001 C CNN "Description"
 F 10 "" H 0   0   50  0001 C CNN "Manufacturer"
+F 11 "C22765" H 650 6650 50  0001 C CNN "LCSC"
 	1    650  6650
 	1    0    0    -1
@@
 F 9 "" H 0   0   50  0001 C CNN "Voltage"
 F 10 "STMicroelectronics" H 0   0   50  0001 C CNN "Manufacturer"
+F 11 "C252436" H 4600 10150 50  0001 C CNN "LCSC"
 	1    4600 10150
 	1    0    0    -1
@@
 F 9 "" H 0   0   50  0001 C CNN "Voltage"
 F 10 "STMicroelectronics" H 0   0   50  0001 C CNN "Manufacturer"
+F 11 "C252436" H 2800 1950 50  0001 C CNN "LCSC"
 	1    2800 1950
 	-1   0    0    -1
@@
 F 9 "" H 0   0   50  0001 C CNN "Voltage"
 F 10 "STMicroelectronics" H 0   0   50  0001 C CNN "Manufacturer"
+F 11 "C252436" H 2800 2650 50  0001 C CNN "LCSC"
 	1    2800 2650
 	-1   0    0    -1
@@
 F 9 "" H 0   0   50  0001 C CNN "Description"
 F 10 "" H 0   0   50  0001 C CNN "Manufacturer"
+F 11 " C14663" H 2150 3450 50  0001 C CNN "LCSC"
 	1    2150 3450
 	1    0    0    -1
@@
 F 9 "" H 0   0   50  0001 C CNN "Description"
 F 10 "" H 0   0   50  0001 C CNN "Manufacturer"
+F 11 " C14663" H 2600 3450 50  0001 C CNN "LCSC"
 	1    2600 3450
 	1    0    0    -1
@@
 F 9 "" H 0   0   50  0001 C CNN "Description"
 F 10 "" H 0   0   50  0001 C CNN "Manufacturer"
+F 11 " C14663" H 4750 9250 50  0001 C CNN "LCSC"
 	1    4750 9250
 	1    0    0    -1
@@
 F 9 "" H 0   0   50  0001 C CNN "Description"
 F 10 "" H 0   0   50  0001 C CNN "Manufacturer"
+F 11 "C21190" H 4950 4000 50  0001 C CNN "LCSC"
 	1    4950 4000
 	0    1    1    0
