File: hw/kicad/v4.0/f4.sch (KiCad schematic (older format))
At the start: 37 parts, among them P1 USB_OTG, U1 USBLC6-4SC6, U20 USBLC6-4SC6, U22 USBLC6-4SC6, U23 USBLC6-4SC6, U26 STM32F405VG, Y2 8M

Commit message: WIP LCSC
Parts:
- C1, C119, C16, C29, C61, C66, C67, C77, C80, C84, C85, C86, C87, C89: LCSC (none) -> C14663
- P1: LCSC (none) -> C145792
- Y2: LCSC (none) -> C389778
Changed lines of the file:
@@
 EESchema Schematic File Version 4
-LIBS:stmbl_4.0-cache
-EELAYER 26 0
+EELAYER 30 0
 EELAYER END
 $Descr A3 16535 11693
@@
 F 9 "" H 0   0   50  0001 C CNN "Description"
 F 10 "Abracon LLC" H 0   0   50  0001 C CNN "Manufacturer"
+F 11 "C389778" H 4700 3700 50  0001 C CNN "LCSC"
 	1    4700 3700
 	0    1    1    0
@@
 F 9 "" H 0   0   50  0001 C CNN "Description"
 F 10 "" H 0   0   50  0001 C CNN "Manufacturer"
+F 11 "C14663" H 11400 2150 50  0001 C CNN "LCSC"
 	1    11400 2150
 	1    0    0    -1
@@
 F 9 "" H 0   0   50  0001 C CNN "Description"
 F 10 "" H 0   0   50  0001 C CNN "Manufacturer"
+F 11 "C14663" H 10900 2150 50  0001 C CNN "LCSC"
 	1    10900 2150
 	1    0    0    -1
@@
 F 9 "" H 0   0   50  0001 C CNN "Description"
 F 10 "" H 0   0   50  0001 C CNN "Manufacturer"
+F 11 "C14663" H 10600 2150 50  0001 C CNN "LCSC"
 	1    10600 2150
 	1    0    0    -1
@@
 F 9 "" H 0   0   50  0001 C CNN "Description"
 F 10 "" H 0   0   50  0001 C CNN "Manufacturer"
+F 11 "C14663" H 10300 2150 50  0001 C CNN "LCSC"
 	1    10300 2150
 	1    0    0    -1
@@
 F 9 "" H 0   0   50  0001 C CNN "Description"
 F 10 "" H 0   0   50  0001 C CNN "Manufacturer"
+F 11 "C14663" H 10000 2150 50  0001 C CNN "LCSC"
 	1    10000 2150
 	1    0    0    -1
@@
 F 9 "" H 0   0   50  0001 C CNN "Description"
 F 10 "" H 0   0   50  0001 C CNN "Manufacturer"
+F 11 "C14663" H 9700 2150 50  0001 C CNN "LCSC"
 	1    9700 2150
 	1    0    0    -1
@@
 F 9 "" H 0   0   50  0001 C CNN "Description"
 F 10 "" H 0   0   50  0001 C CNN "Manufacturer"
+F 11 "C14663" H 9400 2150 50  0001 C CNN "LCSC"
 	1    9400 2150
 	1    0    0    -1
@@
 F 9 "" H 0   0   50  0001 C CNN "Description"
 F 10 "" H 0   0   50  0001 C CNN "Manufacturer"
+F 11 "C14663" H 4600 2850 50  0001 C CNN "LCSC"
 	1    4600 2850
 	1    0    0    -1
@@
 F 9 "" H 0   0   50  0001 C CNN "Description"
 F 10 "Molex" H 0   0   50  0001 C CNN "Manufacturer"
+F 11 "C145792" H 850 6000 50  0001 C CNN "LCSC"
 	1    850  6000
 	0    -1   1    0
@@
 F 9 "" H 0   0   50  0001 C CNN "Description"
 F 10 "" H 0   0   50  0001 C CNN "Manufacturer"
+F 11 "C14663" H 2800 7050 50  0001 C CNN "LCSC"
 	1    2800 7050
 	0    1    1    0
@@
 F 9 "" H 0   0   50  0001 C CNN "Description"
 F 10 "" H 0   0   50  0001 C CNN "Manufacturer"
+F 11 "C14663" H 8100 2150 50  0001 C CNN "LCSC"
 	1    8100 2150
 	1    0    0    -1
@@
 F 9 "" H 0   0   50  0001 C CNN "Description"
 F 10 "" H 0   0   50  0001 C CNN "Manufacturer"
+F 11 "C14663" H 850 6650 50  0001 C CNN "LCSC"
 	1    850  6650
 	1    0    0    -1
@@
 F 9 "" H 0   0   50  0001 C CNN "Description"
 F 10 "" H 0   0   50  0001 C CNN "Manufacturer"
+F 11 "C14663" H 2150 3450 50  0001 C CNN "LCSC"
 	1    2150 3450
 	1    0    0    -1
@@
 F 9 "" H 0   0   50  0001 C CNN "Description"
 F 10 "" H 0   0   50  0001 C CNN "Manufacturer"
+F 11 "C14663" H 2600 3450 50  0001 C CNN "LCSC"
 	1    2600 3450
 	1    0    0    -1
@@
 F 9 "" H 0   0   50  0001 C CNN "Description"
 F 10 "" H 0   0   50  0001 C CNN "Manufacturer"
+F 11 "C14663" H 4750 9250 50  0001 C CNN "LCSC"
 	1    4750 9250
 	1    0    0    -1
