File: hw/kicad/v4.0/fb.sch (KiCad schematic (older format))
At the start: 48 parts, among them J1 RJ45_LED, U15 SN65176B, U16 SN65176B, U19 SN65176B, U7 LM358

Commit message: Added LCSC # to parts in 4.3 PCB
Parts:
- C116, C117, C118, C12, C125, C37, C71, C73, C76: LCSC (none) -> C14663
- C24, C26: LCSC (none) -> C1647
- C46, C49: LCSC (none) -> C1588
- L11, L8: LCSC (none) -> C85827
- R110, R112, R113, R130, R23, R26: LCSC (none) -> C22765
- R124, R125, R128, R136: LCSC (none) -> C21190
- R135, R137, R37, R38, R41, R43: LCSC (none) -> C25804
- R147, R87, R88: LCSC (none) -> C23345
- R4, R5, R94, R96: LCSC (none) -> C23179
- R48, R49, R54, R57: LCSC (none) -> C22809
- U15, U16, U19: LCSC (none) -> C31302
- U7: LCSC (none) -> C74525
Changed lines of the file:
@@
 EESchema Schematic File Version 4
 LIBS:stmbl_4.0-cache
-EELAYER 26 0
+EELAYER 30 0
 EELAYER END
 $Descr A4 11693 8268
@@
 F 9 "" H 0   0   50  0001 C CNN "Description"
 F 10 "Texas Instruments" H 0   0   50  0001 C CNN "Manufacturer"
+F 11 "C74525" H 5000 4500 50  0001 C CNN "LCSC"
 	1    5000 4500
 	1    0    0    -1
@@
 F 9 "" H 0   0   50  0001 C CNN "Description"
 F 10 "Texas Instruments" H 0   0   50  0001 C CNN "Manufacturer"
+F 11 "C31302" H 8150 1250 50  0001 C CNN "LCSC"
 	1    8150 1250
 	-1   0    0    -1
@@
 F 9 "" H 0   0   50  0001 C CNN "Description"
 F 10 "" H 0   0   50  0001 C CNN "Manufacturer"
+F 11 "C22765" H 7600 1250 50  0001 C CNN "LCSC"
 	1    7600 1250
 	1    0    0    -1
@@
 F 9 "" H 0   0   50  0001 C CNN "Description"
 F 10 "" H 0   0   50  0001 C CNN "Manufacturer"
+F 11 " C14663" H 9200 1250 50  0001 C CNN "LCSC"
 	1    9200 1250
 	1    0    0    -1
@@
 F 9 "" H 0   0   50  0001 C CNN "Description"
 F 10 "Texas Instruments" H 0   0   50  0001 C CNN "Manufacturer"
+F 11 "C31302" H 8150 2650 50  0001 C CNN "LCSC"
 	1    8150 2650
 	-1   0    0    -1
@@
 F 9 "" H 0   0   50  0001 C CNN "Description"
 F 10 "" H 0   0   50  0001 C CNN "Manufacturer"
+F 11 "C22765" H 7600 2650 50  0001 C CNN "LCSC"
 	1    7600 2650
 	1    0    0    -1
@@
 F 9 "" H 0   0   50  0001 C CNN "Description"
 F 10 "" H 0   0   50  0001 C CNN "Manufacturer"
+F 11 " C14663" H 9200 2650 50  0001 C CNN "LCSC"
 	1    9200 2650
 	1    0    0    -1
@@
 F 9 "" H 0   0   50  0001 C CNN "Description"
 F 10 "Texas Instruments" H 0   0   50  0001 C CNN "Manufacturer"
+F 11 "C31302" H 8150 4050 50  0001 C CNN "LCSC"
 	1    8150 4050
 	-1   0    0    -1
@@
 F 9 "" H 0   0   50  0001 C CNN "Description"
 F 10 "" H 0   0   50  0001 C CNN "Manufacturer"
+F 11 "C22765" H 7600 4050 50  0001 C CNN "LCSC"
 	1    7600 4050
 	1    0    0    -1
@@
 F 9 "" H 0   0   50  0001 C CNN "Description"
 F 10 "" H 0   0   50  0001 C CNN "Manufacturer"
+F 11 " C14663" H 9200 4050 50  0001 C CNN "LCSC"
 	1    9200 4050
 	1    0    0    -1
@@
 F 9 "" H 0   0   50  0001 C CNN "Description"
 F 10 "" H 0   0   50  0001 C CNN "Manufacturer"
+F 11 "C23179" H 1000 3050 50  0001 C CNN "LCSC"
 	1    1000 3050
 	0    1    1    0
@@
 F 9 "" H 0   0   50  0001 C CNN "Description"
 F 10 "" H 0   0   50  0001 C CNN "Manufacturer"
+F 11 "C23179" H 1000 3750 50  0001 C CNN "LCSC"
 	1    1000 3750
 	0    1    1    0
@@
 F 9 "" H 0   0   50  0001 C CNN "Description"
 F 10 "" H 0   0   50  0001 C CNN "Manufacturer"
+F 11 "C25804" H 4150 4350 50  0001 C CNN "LCSC"
 	1    4150 4350
 	0    1    1    0
@@
 F 9 "" H 0   0   50  0001 C CNN "Description"
 F 10 "" H 0   0   50  0001 C CNN "Manufacturer"
+F 11 "C25804" H 4150 4650 50  0001 C CNN "LCSC"
 	1    4150 4650
 	0    1    1    0
@@
 F 9 "" H 0   0   50  0001 C CNN "Description"
 F 10 "" H 0   0   50  0001 C CNN "Manufacturer"
+F 11 "C22809" H 4350 4100 50  0001 C CNN "LCSC"
 	1    4350 4100
 	1    0    0    -1
@@
 F 9 "" H 0   0   50  0001 C CNN "Description"
 F 10 "" H 0   0   50  0001 C CNN "Manufacturer"
+F 11 "C22809" H 4600 4850 50  0001 C CNN "LCSC"
 	1    4600 4850
 	0    1    1    0
@@
 F 9 "" H 0   0   50  0001 C CNN "Description"
 F 10 "" H 0   0   50  0001 C CNN "Manufacturer"
+F 11 "C23345" H 5850 4500 50  0001 C CNN "LCSC"
 	1    5850 4500
 	0    1    1    0
@@
 F 9 "" H 0   0   50  0001 C CNN "Description"
 F 10 "" H 0   0   50  0001 C CNN "Manufacturer"
+F 11 "C23179" H 6200 4750 50  0001 C CNN "LCSC"
 	1    6200 4750
 	1    0    0    -1
@@
 F 9 "" H 0   0   50  0001 C CNN "Description"
 F 10 "" H 0   0   50  0001 C CNN "Manufacturer"
+F 11 "C1588" H 6000 4750 50  0001 C CNN "LCSC"
 	1    6000 4750
 	1    0    0    -1
@@
 F 9 "" H 0   0   50  0001 C CNN "Description"
 F 10 "" H 0   0   50  0001 C CNN "Manufacturer"
+F 11 "C25804" H 4050 5450 50  0001 C CNN "LCSC"
 	1    4050 5450
 	0    1    1    0
@@
 F 9 "" H 0   0   50  0001 C CNN "Description"
 F 10 "" H 0   0   50  0001 C CNN "Manufacturer"
+F 11 "C25804" H 4050 5750 50  0001 C CNN "LCSC"
 	1    4050 5750
 	0    1    1    0
@@
 F 9 "" H 0   0   50  0001 C CNN "Description"
 F 10 "" H 0   0   50  0001 C CNN "Manufacturer"
+F 11 "C22809" H 4300 5200 50  0001 C CNN "LCSC"
 	1    4300 5200
 	1    0    0    -1
@@
 F 9 "" H 0   0   50  0001 C CNN "Description"
 F 10 "" H 0   0   50  0001 C CNN "Manufacturer"
+F 11 "C22809" H 4600 5950 50  0001 C CNN "LCSC"
 	1    4600 5950
 	0    1    1    0
@@
 F 9 "" H 0   0   50  0001 C CNN "Description"
 F 10 "" H 0   0   50  0001 C CNN "Manufacturer"
+F 11 "C23345" H 5850 5600 50  0001 C CNN "LCSC"
 	1    5850 5600
 	0    1    1    0
@@
 F 9 "" H 0   0   50  0001 C CNN "Description"
 F 10 "" H 0   0   50  0001 C CNN "Manufacturer"
+F 11 "C23179" H 6200 5850 50  0001 C CNN "LCSC"
 	1    6200 5850
 	1    0    0    -1
@@
 F 9 "" H 0   0   50  0001 C CNN "Description"
 F 10 "" H 0   0   50  0001 C CNN "Manufacturer"
+F 11 "C1588" H 6000 5850 50  0001 C CNN "LCSC"
 	1    6000 5850
 	1    0    0    -1
@@
 F 9 "" H 0   0   50  0001 C CNN "Description"
 F 10 "" H 0   0   50  0001 C CNN "Manufacturer"
+F 11 "C22765" H 2500 5900 50  0001 C CNN "LCSC"
 	1    2500 5900
 	1    0    0    -1
@@
 F 9 "" H 0   0   50  0001 C CNN "Description"
 F 10 "" H 0   0   50  0001 C CNN "Manufacturer"
+F 11 "C22765" H 2500 6800 50  0001 C CNN "LCSC"
 	1    2500 6800
 	1    0    0    -1
@@
 F 9 "" H 0   0   50  0001 C CNN "Description"
 F 10 "" H 0   0   50  0001 C CNN "Manufacturer"
+F 11 " C14663" H 2700 6800 50  0001 C CNN "LCSC"
 	1    2700 6800
 	1    0    0    -1
@@
 F 9 "" H 0   0   50  0001 C CNN "Description"
 F 10 "" H 0   0   50  0001 C CNN "Manufacturer"
+F 11 " C14663" H 3100 5750 50  0001 C CNN "LCSC"
 	1    3100 5750
 	-1   0    0    1
@@
 F 9 "" H 0   0   50  0001 C CNN "Description"
 F 10 "" H 0   0   50  0001 C CNN "Manufacturer"
+F 11 "C1647" H 4300 5600 50  0001 C CNN "LCSC"
 	1    4300 5600
 	1    0    0    -1
@@
 F 9 "" H 0   0   50  0001 C CNN "Description"
 F 10 "" H 0   0   50  0001 C CNN "Manufacturer"
+F 11 "C1647" H 4350 4500 50  0001 C CNN "LCSC"
 	1    4350 4500
 	1    0    0    -1
@@
 F 9 "" H 0   0   50  0001 C CNN "Description"
 F 10 "" H 0   0   50  0001 C CNN "Manufacturer"
+F 11 "C21190" H 9550 1450 50  0001 C CNN "LCSC"
 	1    9550 1450
 	1    0    0    -1
@@
 F 9 "" H 0   0   50  0001 C CNN "Description"
 F 10 "" H 0   0   50  0001 C CNN "Manufacturer"
+F 11 "C21190" H 9550 2850 50  0001 C CNN "LCSC"
 	1    9550 2850
 	1    0    0    -1
@@
 F 9 "" H 0   0   50  0001 C CNN "Description"
 F 10 "" H 0   0   50  0001 C CNN "Manufacturer"
+F 11 "C21190" H 9550 4250 50  0001 C CNN "LCSC"
 	1    9550 4250
 	1    0    0    -1
@@
 F 9 "" H 0   0   50  0001 C CNN "Description"
 F 10 "Murata" H 0   0   50  0001 C CNN "Manufacturer"
+F 11 "C85827" H 2100 5250 50  0001 C CNN "LCSC"
 	1    2100 5250
 	0    -1   -1   0
@@
 F 9 "" H 0   0   50  0001 C CNN "Description"
 F 10 "" H 0   0   50  0001 C CNN "Manufacturer"
+F 11 " C14663" H 1700 5500 50  0001 C CNN "LCSC"
 	1    1700 5500
 	-1   0    0    1
@@
 F 9 "" H 0   0   50  0001 C CNN "Description"
 F 10 "Murata" H 0   0   50  0001 C CNN "Manufacturer"
+F 11 "C85827" H 10300 800 50  0001 C CNN "LCSC"
 	1    10300 800
 	0    1    -1   0
@@
 F 9 "" H 0   0   50  0001 C CNN "Description"
 F 10 "" H 0   0   50  0001 C CNN "Manufacturer"
+F 11 " C14663" H 10700 1050 50  0001 C CNN "LCSC"
 	1    10700 1050
 	1    0    0    1
@@
 F 9 "" H 0   0   50  0001 C CNN "Description"
 F 10 "" H 0   0   50  0001 C CNN "Manufacturer"
+F 11 "C22765" H 2500 5500 50  0001 C CNN "LCSC"
 	1    2500 5500
 	1    0    0    -1
@@
 F 9 "" H 0   0   50  0001 C CNN "Description"
 F 10 "" H 0   0   50  0001 C CNN "Manufacturer"
+F 11 " C14663" H 2500 3900 50  0001 C CNN "LCSC"
 	1    2500 3900
 	1    0    0    -1
@@
 F 9 "" H 0   0   50  0001 C CNN "Description"
 F 10 "" H 0   0   50  0001 C CNN "Manufacturer"
+F 11 "C25804" H 2950 4250 50  0001 C CNN "LCSC"
 	1    2950 4250
 	1    0    0    -1
@@
 F 9 "" H 0   0   50  0001 C CNN "Description"
 F 10 "" H 0   0   50  0001 C CNN "Manufacturer"
+F 11 "C25804" H 2750 4250 50  0001 C CNN "LCSC"
 	1    2750 4250
 	1    0    0    -1
@@
 F 9 "" H 0   0   50  0001 C CNN "Description"
 F 10 "" H 0   0   50  0001 C CNN "Manufacturer"
+F 11 "C21190" H 2750 4750 50  0001 C CNN "LCSC"
 	1    2750 4750
 	1    0    0    -1
@@
 F 9 "" H 0   0   50  0001 C CNN "Description"
 F 10 "" H 0   0   50  0001 C CNN "Manufacturer"
+F 11 " C14663" H 2450 4750 50  0001 C CNN "LCSC"
 	1    2450 4750
 	1    0    0    -1
@@
 F 9 "" H 0   0   50  0001 C CNN "Description"
 F 10 "Texas Instruments" H 0   0   50  0001 C CNN "Manufacturer"
+F 11 "C74525" H 5000 5600 50  0001 C CNN "LCSC"
 	2    5000 5600
 	1    0    0    -1
@@
 F 9 "" H 0   0   50  0001 C CNN "Description"
 F 10 "" H 0   0   50  0001 C CNN "Manufacturer"
+F 11 "C23345" H 2500 6400 50  0001 C CNN "LCSC"
 	1    2500 6400
 	1    0    0    -1
