File: hw/kicad/v4.0/fb.sch (KiCad schematic (older format))
At the start: 48 parts, among them J1 RJ45_LED, U15 SN65176B, U16 SN65176B, U19 SN65176B, U7 LM358

Commit message: WIP LCSC
Parts:
- C116, C117, C118, C12, C125, C37, C71, C73, C76: LCSC (none) -> C14663
- J1: LCSC (none) -> C138392
Changed lines of the file:
@@
 EESchema Schematic File Version 4
-LIBS:stmbl_4.0-cache
-EELAYER 26 0
+EELAYER 30 0
 EELAYER END
 $Descr A4 11693 8268
@@
 F 9 "" H 0   0   50  0001 C CNN "Description"
 F 10 "METZ CONNECT" H 0   0   50  0001 C CNN "Manufacturer"
+F 11 "C138392" H 1700 3350 50  0001 C CNN "LCSC"
 	1    1700 3350
 	0    -1   1    0
@@
 F 9 "" H 0   0   50  0001 C CNN "Description"
 F 10 "" H 0   0   50  0001 C CNN "Manufacturer"
+F 11 "C14663" H 9200 1250 50  0001 C CNN "LCSC"
 	1    9200 1250
 	1    0    0    -1
@@
 F 9 "" H 0   0   50  0001 C CNN "Description"
 F 10 "" H 0   0   50  0001 C CNN "Manufacturer"
+F 11 "C14663" H 9200 2650 50  0001 C CNN "LCSC"
 	1    9200 2650
 	1    0    0    -1
@@
 F 9 "" H 0   0   50  0001 C CNN "Description"
 F 10 "" H 0   0   50  0001 C CNN "Manufacturer"
+F 11 "C14663" H 9200 4050 50  0001 C CNN "LCSC"
 	1    9200 4050
 	1    0    0    -1
@@
 F 9 "" H 0   0   50  0001 C CNN "Description"
 F 10 "" H 0   0   50  0001 C CNN "Manufacturer"
+F 11 "C14663" H 2700 6800 50  0001 C CNN "LCSC"
 	1    2700 6800
 	1    0    0    -1
@@
 F 9 "" H 0   0   50  0001 C CNN "Description"
 F 10 "" H 0   0   50  0001 C CNN "Manufacturer"
+F 11 "C14663" H 3100 5750 50  0001 C CNN "LCSC"
 	1    3100 5750
 	-1   0    0    1
@@
 F 9 "" H 0   0   50  0001 C CNN "Description"
 F 10 "" H 0   0   50  0001 C CNN "Manufacturer"
+F 11 "C14663" H 1700 5500 50  0001 C CNN "LCSC"
 	1    1700 5500
 	-1   0    0    1
@@
 F 9 "" H 0   0   50  0001 C CNN "Description"
 F 10 "" H 0   0   50  0001 C CNN "Manufacturer"
+F 11 "C14663" H 10700 1050 50  0001 C CNN "LCSC"
 	1    10700 1050
 	1    0    0    1
@@
 F 9 "" H 0   0   50  0001 C CNN "Description"
 F 10 "" H 0   0   50  0001 C CNN "Manufacturer"
+F 11 "C14663" H 2500 3900 50  0001 C CNN "LCSC"
 	1    2500 3900
 	1    0    0    -1
@@
 F 9 "" H 0   0   50  0001 C CNN "Description"
 F 10 "" H 0   0   50  0001 C CNN "Manufacturer"
+F 11 "C14663" H 2450 4750 50  0001 C CNN "LCSC"
 	1    2450 4750
 	1    0    0    -1
