File: hw/kicad/v4.0/hv.sch (KiCad schematic (older format))
At the start: 21 parts, among them P13 CONN_01X04, P2 CONN_01X02, Q5 IRLML6344, U24 non_plated, U3 SI8621, U30 non_plated, U31 non_plated

Commit message: Added LCSC # to parts in 4.3 PCB
Parts:
- C127, C138, C19, C30, C40: LCSC (none) -> C14663
- Q5: LCSC (none) -> C53550
- R141: LCSC (none) -> C23196
- R142, R7: LCSC (none) -> C25804
- R162, R165: LCSC (none) -> C21190
- R163, R167: LCSC (none) -> C23345
- R164, R166: LCSC (none) -> C23018
Changed lines of the file:
@@
 EESchema Schematic File Version 4
 LIBS:stmbl_4.0-cache
-EELAYER 26 0
+EELAYER 30 0
 EELAYER END
 $Descr A4 11693 8268
@@
 F 9 "" H 0   0   50  0001 C CNN "InternalName"
 F 10 "" H 0   0   50  0001 C CNN "Manufacturer"
+F 11 " C14663" H 3450 1150 50  0001 C CNN "LCSC"
 	1    3450 1150
 	0    1    1    0
@@
 F 9 "" H 0   0   50  0001 C CNN "InternalName"
 F 10 "" H 0   0   50  0001 C CNN "Manufacturer"
+F 11 " C14663" H 4650 1150 50  0001 C CNN "LCSC"
 	1    4650 1150
 	0    1    1    0
@@
 F 9 "" H 50  -300 50  0001 C CNN "InternalName"
 F 10 "" H 50  -300 50  0001 C CNN "Manufacturer"
+F 11 "C25804" H 9950 1100 50  0001 C CNN "LCSC"
 	1    9950 1100
 	1    0    0    -1
@@
 F 9 "" H -350 0   50  0001 C CNN "InternalName"
 F 10 "" H -350 0   50  0001 C CNN "Manufacturer"
+F 11 " C14663" H 8450 1900 50  0001 C CNN "LCSC"
 	1    8450 1900
 	-1   0    0    1
@@
 F 9 "" H -400 -200 50  0001 C CNN "Voltage"
 F 10 "" H -400 -200 50  0001 C CNN "Manufacturer"
+F 11 "C23196" H 9250 1450 50  0001 C CNN "LCSC"
 	1    9250 1450
 	0    1    1    0
@@
 F 9 "" H -400 0   50  0001 C CNN "InternalName"
 F 10 "" H -400 0   50  0001 C CNN "Manufacturer"
+F 11 "C25804" H 8700 1900 50  0001 C CNN "LCSC"
 	1    8700 1900
 	-1   0    0    1
@@
 F 9 "" H -400 0   50  0001 C CNN "InternalName"
 F 10 "" H -400 0   50  0001 C CNN "Manufacturer"
+F 11 " C14663" H 9000 1900 50  0001 C CNN "LCSC"
 	1    9000 1900
 	-1   0    0    1
@@
 F 9 "" H 500 0   50  0001 C CNN "InternalName"
 F 10 "" H 500 0   50  0001 C CNN "Manufacturer"
+F 11 " C14663" H 11100 1900 50  0001 C CNN "LCSC"
 	1    11100 1900
 	-1   0    0    1
@@
 F 9 "" H 0   0   50  0001 C CNN "InternalName"
 F 10 "" H 0   0   50  0001 C CNN "Manufacturer"
+F 11 "C21190" H 8450 2600 50  0001 C CNN "LCSC"
 	1    8450 2600
 	0    -1   -1   0
@@
 F 9 "" H 8150 -2000 50  0001 C CNN "Description"
 F 10 "Infineon" H 8150 -2000 50  0001 C CNN "Manufacturer"
+F 11 "C53550" H 10150 1850 50  0001 C CNN "LCSC"
 	1    10150 1850
 	1    0    0    -1
@@
 F 9 "" H 7800 -2250 50  0001 C CNN "Description"
 F 10 "" H 7800 -2250 50  0001 C CNN "Manufacturer"
+F 11 "C23345" H 9250 1650 50  0001 C CNN "LCSC"
 	1    9250 1650
 	0    -1   -1   0
@@
 F 9 "" H 7900 -3050 50  0001 C CNN "Description"
 F 10 "" H 7900 -3050 50  0001 C CNN "Manufacturer"
+F 11 "C23018" H 9600 1100 50  0001 C CNN "LCSC"
 	1    9600 1100
 	1    0    0    -1
@@
 F 9 "" H 7900 -2250 50  0001 C CNN "Description"
 F 10 "" H 7900 -2250 50  0001 C CNN "Manufacturer"
+F 11 "C21190" H 9600 1900 50  0001 C CNN "LCSC"
 	1    9600 1900
 	1    0    0    -1
@@
 F 9 "" H 350 -300 50  0001 C CNN "InternalName"
 F 10 "" H 350 -300 50  0001 C CNN "Manufacturer"
+F 11 "C23018" H 10250 1100 50  0001 C CNN "LCSC"
 	1    10250 1100
 	1    0    0    -1
@@
 F 9 "" H 9050 -2350 50  0001 C CNN "Description"
 F 10 "" H 9050 -2350 50  0001 C CNN "Manufacturer"
+F 11 "C23345" H 10500 1550 50  0001 C CNN "LCSC"
 	1    10500 1550
 	0    -1   -1   0
