File: hw/kicad/v4.0/hv.sch (KiCad schematic (older format))
At the start: 21 parts, among them P13 CONN_01X04, P2 CONN_01X02, Q5 IRLML6344, U24 non_plated, U3 SI8621, U30 non_plated, U31 non_plated

Commit message: WIP LCSC
Parts:
- C127, C138, C19, C30, C40: LCSC (none) -> C14663
- P2: LCSC (none) -> C441171
Changed lines of the file:
@@
 EESchema Schematic File Version 4
-LIBS:stmbl_4.0-cache
-EELAYER 26 0
+EELAYER 30 0
 EELAYER END
 $Descr A4 11693 8268
@@
 F 9 "" H 0   0   50  0001 C CNN "InternalName"
 F 10 "" H 0   0   50  0001 C CNN "Manufacturer"
+F 11 "C14663" H 3450 1150 50  0001 C CNN "LCSC"
 	1    3450 1150
 	0    1    1    0
@@
 F 9 "" H 0   0   50  0001 C CNN "InternalName"
 F 10 "" H 0   0   50  0001 C CNN "Manufacturer"
+F 11 "C14663" H 4650 1150 50  0001 C CNN "LCSC"
 	1    4650 1150
 	0    1    1    0
@@
 F 9 "" H 750 -200 50  0001 C CNN "InternalName"
 F 10 "Phoenix" H 750 -200 50  0001 C CNN "Manufacturer"
+F 11 "C441171" H 10950 1500 50  0001 C CNN "LCSC"
 	1    10950 1500
 	1    0    0    -1
@@
 F 9 "" H -350 0   50  0001 C CNN "InternalName"
 F 10 "" H -350 0   50  0001 C CNN "Manufacturer"
+F 11 "C14663" H 8450 1900 50  0001 C CNN "LCSC"
 	1    8450 1900
 	-1   0    0    1
@@
 F 9 "" H -400 0   50  0001 C CNN "InternalName"
 F 10 "" H -400 0   50  0001 C CNN "Manufacturer"
+F 11 "C14663" H 9000 1900 50  0001 C CNN "LCSC"
 	1    9000 1900
 	-1   0    0    1
@@
 F 9 "" H 500 0   50  0001 C CNN "InternalName"
 F 10 "" H 500 0   50  0001 C CNN "Manufacturer"
+F 11 "C14663" H 11100 1900 50  0001 C CNN "LCSC"
 	1    11100 1900
 	-1   0    0    1
