File: hw/kicad/v4.0/hv.sch (KiCad schematic (older format))
At the start: 21 parts, among them P13 CONN_01X04, P2 CONN_01X02, Q5 IRLML6344, U24 non_plated, U3 SI8621, U30 non_plated, U31 non_plated

Commit message: Changed 120uf 1808 to 1210 100uF
Parts:
- C127, C138, C19, C30, C40: LCSC C14663 -> C14663
Changed lines of the file:
@@
 F 9 "" H 0   0   50  0001 C CNN "InternalName"
 F 10 "" H 0   0   50  0001 C CNN "Manufacturer"
-F 11 " C14663" H 3450 1150 50  0001 C CNN "LCSC"
+F 11 "C14663" H 3450 1150 50  0001 C CNN "LCSC"
 	1    3450 1150
 	0    1    1    0
@@
 F 9 "" H 0   0   50  0001 C CNN "InternalName"
 F 10 "" H 0   0   50  0001 C CNN "Manufacturer"
-F 11 " C14663" H 4650 1150 50  0001 C CNN "LCSC"
+F 11 "C14663" H 4650 1150 50  0001 C CNN "LCSC"
 	1    4650 1150
 	0    1    1    0
@@
 F 9 "" H -350 0   50  0001 C CNN "InternalName"
 F 10 "" H -350 0   50  0001 C CNN "Manufacturer"
-F 11 " C14663" H 8450 1900 50  0001 C CNN "LCSC"
+F 11 "C14663" H 8450 1900 50  0001 C CNN "LCSC"
 	1    8450 1900
 	-1   0    0    1
@@
 F 9 "" H -400 0   50  0001 C CNN "InternalName"
 F 10 "" H -400 0   50  0001 C CNN "Manufacturer"
-F 11 " C14663" H 9000 1900 50  0001 C CNN "LCSC"
+F 11 "C14663" H 9000 1900 50  0001 C CNN "LCSC"
 	1    9000 1900
 	-1   0    0    1
@@
 F 9 "" H 500 0   50  0001 C CNN "InternalName"
 F 10 "" H 500 0   50  0001 C CNN "Manufacturer"
-F 11 " C14663" H 11100 1900 50  0001 C CNN "LCSC"
+F 11 "C14663" H 11100 1900 50  0001 C CNN "LCSC"
 	1    11100 1900
 	-1   0    0    1

Commit message: Switch some 2.2uf 0603 to 1uf bypass to get 50V version on jlcpcb
Change 2.2uf 0603 to 0805 on iram to get 50V version on jlcpcb
other cleanup
Parts:
- C127, C138, C19, C30, C40: Manufacturer (none) -> YAGEO; Manufacturer No (none) -> CC0603KRX7R9BB104
- P2: LCSC C441171 -> (none)
Changed lines of the file:
@@
 F 2 "stmbl:C_0603" H 3488 1000 30  0001 C CNN
 F 3 "" H 3450 1150 60  0000 C CNN
-F 4 "" H 3450 1150 50  0001 C CNN "Manufacturer No"
+F 4 "CC0603KRX7R9BB104 " H 3450 1150 50  0001 C CNN "Manufacturer No"
 F 5 "50V" H 3450 1150 50  0001 C CNN "Voltage"
 F 6 "" H 3450 1150 50  0001 C CNN "Source"
@@
 F 8 "" H 0   0   50  0001 C CNN "Description"
 F 9 "" H 0   0   50  0001 C CNN "InternalName"
-F 10 "" H 0   0   50  0001 C CNN "Manufacturer"
+F 10 "YAGEO" H 0   0   50  0001 C CNN "Manufacturer"
 F 11 "C14663" H 3450 1150 50  0001 C CNN "LCSC"
 	1    3450 1150
@@
 F 2 "stmbl:C_0603" H 4688 1000 30  0001 C CNN
 F 3 "" H 4650 1150 60  0000 C CNN
-F 4 "" H 4650 1150 50  0001 C CNN "Manufacturer No"
+F 4 "CC0603KRX7R9BB104 " H 4650 1150 50  0001 C CNN "Manufacturer No"
 F 5 "50V" H 4650 1150 50  0001 C CNN "Voltage"
 F 6 "" H 4650 1150 50  0001 C CNN "Source"
@@
 F 8 "" H 0   0   50  0001 C CNN "Description"
 F 9 "" H 0   0   50  0001 C CNN "InternalName"
-F 10 "" H 0   0   50  0001 C CNN "Manufacturer"
+F 10 "YAGEO" H 0   0   50  0001 C CNN "Manufacturer"
 F 11 "C14663" H 4650 1150 50  0001 C CNN "LCSC"
 	1    4650 1150
@@
 F 9 "" H 0   0   50  0001 C CNN "Voltage"
 F 10 "" H 0   0   50  0001 C CNN "Manufacturer"
+F 11 "" H 2300 1750 50  0001 C CNN "LCSC"
 	1    2300 1750
 	-1   0    0    1
@@
 F 9 "" H 750 -200 50  0001 C CNN "InternalName"
 F 10 "Phoenix" H 750 -200 50  0001 C CNN "Manufacturer"
-F 11 "C441171" H 10950 1500 50  0001 C CNN "LCSC"
+F 11 "" H 10950 1500 50  0001 C CNN "LCSC"
 	1    10950 1500
 	1    0    0    -1
@@
 F 2 "stmbl:C_0603" H 8488 1750 30  0001 C CNN
 F 3 "" H 8450 1900 60  0000 C CNN
-F 4 "" H 8450 1900 50  0001 C CNN "Manufacturer No"
+F 4 "CC0603KRX7R9BB104 " H 8450 1900 50  0001 C CNN "Manufacturer No"
 F 5 "50V" H 8450 1900 50  0001 C CNN "Voltage"
 F 6 "" H 8450 1900 50  0001 C CNN "Source"
@@
 F 8 "" H -350 0   50  0001 C CNN "Description"
 F 9 "" H -350 0   50  0001 C CNN "InternalName"
-F 10 "" H -350 0   50  0001 C CNN "Manufacturer"
+F 10 "YAGEO" H -350 0   50  0001 C CNN "Manufacturer"
 F 11 "C14663" H 8450 1900 50  0001 C CNN "LCSC"
 	1    8450 1900
@@
 F 2 "stmbl:C_0603" H 9038 1750 30  0001 C CNN
 F 3 "" H 9000 1900 60  0000 C CNN
-F 4 "" H 9000 1900 50  0001 C CNN "Manufacturer No"
+F 4 "CC0603KRX7R9BB104 " H 9000 1900 50  0001 C CNN "Manufacturer No"
 F 5 "50V" H 9000 1900 50  0001 C CNN "Voltage"
 F 6 "" H 9000 1900 50  0001 C CNN "Source"
@@
 F 8 "" H -400 0   50  0001 C CNN "Description"
 F 9 "" H -400 0   50  0001 C CNN "InternalName"
-F 10 "" H -400 0   50  0001 C CNN "Manufacturer"
+F 10 "YAGEO" H -400 0   50  0001 C CNN "Manufacturer"
 F 11 "C14663" H 9000 1900 50  0001 C CNN "LCSC"
 	1    9000 1900
@@
 F 2 "stmbl:C_0603" H 11138 1750 30  0001 C CNN
 F 3 "" H 11100 1900 60  0000 C CNN
-F 4 "" H 11100 1900 50  0001 C CNN "Manufacturer No"
+F 4 "CC0603KRX7R9BB104 " H 11100 1900 50  0001 C CNN "Manufacturer No"
 F 5 "50V" H 11100 1900 50  0001 C CNN "Voltage"
 F 6 "" H 11100 1900 50  0001 C CNN "Source"
@@
 F 8 "" H 500 0   50  0001 C CNN "Description"
 F 9 "" H 500 0   50  0001 C CNN "InternalName"
-F 10 "" H 500 0   50  0001 C CNN "Manufacturer"
+F 10 "YAGEO" H 500 0   50  0001 C CNN "Manufacturer"
 F 11 "C14663" H 11100 1900 50  0001 C CNN "LCSC"
 	1    11100 1900
