File: hw/kicad/v4.0/hv_drive.sch (KiCad schematic (older format))
At the start: 21 parts, among them P6 CONN_01X02, P8 CONN_01X03, U12 IRAM256a

Commit message: Added LCSC # to parts in 4.3 PCB
Parts:
- C129, C42, C43, C44: LCSC (none) -> C23630
- C14: LCSC (none) -> C15850
- C147, C63: LCSC (none) -> C14663
- R115: LCSC (none) -> C25804
- R80, R81, R82: LCSC (none) -> C60922
Changed lines of the file:
@@
 EESchema Schematic File Version 4
 LIBS:stmbl_4.0-cache
-EELAYER 26 0
+EELAYER 30 0
 EELAYER END
 $Descr A4 11693 8268
@@
 F 9 "" H 0   0   50  0001 C CNN "Description"
 F 10 "" H 0   0   50  0001 C CNN "Manufacturer"
+F 11 "C23630" H 5600 3050 50  0001 C CNN "LCSC"
 	1    5600 3050
 	0    -1   -1   0
@@
 F 9 "" H 0   0   50  0001 C CNN "Description"
 F 10 "" H 0   0   50  0001 C CNN "Manufacturer"
+F 11 "C23630" H 5600 3450 50  0001 C CNN "LCSC"
 	1    5600 3450
 	0    -1   -1   0
@@
 F 9 "" H 0   0   50  0001 C CNN "Description"
 F 10 "" H 0   0   50  0001 C CNN "Manufacturer"
+F 11 "C23630" H 5600 3850 50  0001 C CNN "LCSC"
 	1    5600 3850
 	0    -1   -1   0
@@
 F 9 "" H 0   0   50  0001 C CNN "Description"
 F 10 "Bourns" H 0   0   50  0001 C CNN "Manufacturer"
+F 11 "C60922" H 5400 4550 50  0001 C CNN "LCSC"
 	1    5400 4550
 	0    1    1    0
@@
 F 9 "" H 0   0   50  0001 C CNN "Description"
 F 10 "Bourns" H 0   0   50  0001 C CNN "Manufacturer"
+F 11 "C60922" H 5400 4750 50  0001 C CNN "LCSC"
 	1    5400 4750
 	0    1    1    0
@@
 F 9 "" H 0   0   50  0001 C CNN "Description"
 F 10 "Bourns" H 0   0   50  0001 C CNN "Manufacturer"
+F 11 "C60922" H 5400 4950 50  0001 C CNN "LCSC"
 	1    5400 4950
 	0    1    1    0
@@
 F 9 "" H 0   0   50  0001 C CNN "Description"
 F 10 "" H 0   0   50  0001 C CNN "Manufacturer"
+F 11 " C14663" H 7800 4900 50  0001 C CNN "LCSC"
 	1    7800 4900
 	1    0    0    -1
@@
 F 9 "" H 0   0   50  0001 C CNN "Description"
 F 10 "" H 0   0   50  0001 C CNN "Manufacturer"
+F 11 "C25804" H 7800 4300 50  0001 C CNN "LCSC"
 	1    7800 4300
 	1    0    0    -1
@@
 F 9 "" H 0   0   50  0001 C CNN "Description"
 F 10 "" H 0   0   50  0001 C CNN "Manufacturer"
+F 11 "C23630" H 8100 4900 50  0001 C CNN "LCSC"
 	1    8100 4900
 	1    0    0    -1
@@
 F 9 "" H 0   0   50  0001 C CNN "Description"
 F 10 "" H 0   0   50  0001 C CNN "Manufacturer"
+F 11 " C15850" H 8400 4900 50  0001 C CNN "LCSC"
 	1    8400 4900
 	1    0    0    1
@@
 F 9 "" H 0   0   50  0001 C CNN "Description"
 F 10 "" H 0   0   50  0001 C CNN "Manufacturer"
+F 11 " C14663" H 8800 4900 50  0001 C CNN "LCSC"
 	1    8800 4900
 	1    0    0    -1
