File: hw/kicad/v4.0/hv_drive.sch (KiCad schematic (older format))
At the start: 21 parts, among them P6 CONN_01X02, P8 CONN_01X03, U12 IRAM256a

Commit message: WIP LCSC
Parts:
- C147, C63: LCSC (none) -> C14663
- P6: LCSC (none) -> C3697
- P8: LCSC (none) -> C8377
Changed lines of the file:
@@
 EESchema Schematic File Version 4
-LIBS:stmbl_4.0-cache
-EELAYER 26 0
+EELAYER 30 0
 EELAYER END
 $Descr A4 11693 8268
@@
 F 9 "" H 0   0   50  0001 C CNN "Description"
 F 10 "" H 0   0   50  0001 C CNN "Manufacturer"
+F 11 "C14663" H 7800 4900 50  0001 C CNN "LCSC"
 	1    7800 4900
 	1    0    0    -1
@@
 F 9 "" H 0   0   50  0001 C CNN "Description"
 F 10 "Phoenix" H 0   0   50  0001 C CNN "Manufacturer"
+F 11 "C8377" H 5450 2000 50  0001 C CNN "LCSC"
 	1    5450 2000
 	1    0    0    -1
@@
 F 9 "" H 0   0   50  0001 C CNN "Description"
 F 10 "Phoenix" H 0   0   50  0001 C CNN "Manufacturer"
+F 11 "C3697" H 3900 1950 50  0001 C CNN "LCSC"
 	1    3900 1950
 	-1   0    0    1
@@
 F 9 "" H 0   0   50  0001 C CNN "Description"
 F 10 "" H 0   0   50  0001 C CNN "Manufacturer"
+F 11 "C14663" H 8800 4900 50  0001 C CNN "LCSC"
 	1    8800 4900
 	1    0    0    -1
