File: hw/kicad/v4.0/supply.sch (KiCad schematic (older format))
At the start: 65 parts, among them P3 CONN_01X02, U13 ACT4088, U2 zldo1117, U27 ACT4088, U28 ACT4088

Commit message: Added LCSC # to parts in 4.3 PCB
Parts:
- C101, C102, C133, C134, C135, C136, C137, C139, C140, C142, C144, C18, C62, C8: LCSC (none) -> C23630
- C103, C104, C105, C106, C107, C108, C120, C121, C122, C96, C99: LCSC (none) -> C14663
- C109, C110, C111, C123, C124, C131, C132: LCSC (none) -> C15850
- D12, D13, D9: LCSC (none) -> C8678
- D22: LCSC (none) -> C10769
- D24: LCSC (none) -> C2297
- R132, R155, R156, R157, R158, R35: LCSC (none) -> C25804
- R133, R60, R97: LCSC (none) -> C23196
- R144, R146, R149, R59: LCSC (none) -> C23018
- R145: LCSC (none) -> C21190
- R154, R159, R160: LCSC (none) -> C23345
- U13, U27, U28: LCSC (none) -> C11135
- U2: LCSC (none) -> C326523
