File: hw/kicad/v4.0/supply.sch (KiCad schematic (older format))
At the start: 65 parts, among them P3 CONN_01X02, U13 ACT4088, U2 zldo1117, U27 ACT4088, U28 ACT4088

Commit message: WIP LCSC
Parts:
- C103, C104, C105, C106, C107, C108, C120, C121, C122, C96, C99: LCSC (none) -> C14663
- P3: LCSC (none) -> C441171
Changed lines of the file:
@@
 EESchema Schematic File Version 4
-LIBS:stmbl_4.0-cache
-EELAYER 26 0
+EELAYER 30 0
 EELAYER END
 $Descr A4 11693 8268
@@
 F 9 "" H 0   0   50  0001 C CNN "Description"
 F 10 "Phoenix" H 0   0   50  0001 C CNN "Manufacturer"
+F 11 "C441171" H 800 3000 50  0001 C CNN "LCSC"
 	1    800  3000
 	-1   0    0    -1
@@
 F 9 "" H 0   0   50  0001 C CNN "Description"
 F 10 "" H 0   0   50  0001 C CNN "Manufacturer"
+F 11 "C14663" H 6850 4800 50  0001 C CNN "LCSC"
 	1    6850 4800
 	0    -1   -1   0
@@
 F 9 "" H 0   0   50  0001 C CNN "Description"
 F 10 "" H 0   0   50  0001 C CNN "Manufacturer"
+F 11 "C14663" H 6850 3000 50  0001 C CNN "LCSC"
 	1    6850 3000
 	0    -1   -1   0
@@
 F 9 "" H 0   0   50  0001 C CNN "Description"
 F 10 "" H 0   0   50  0001 C CNN "Manufacturer"
+F 11 "C14663" H 1200 5350 50  0001 C CNN "LCSC"
 	1    1200 5350
 	1    0    0    -1
@@
 F 9 "" H 0   0   50  0001 C CNN "Description"
 F 10 "" H 0   0   50  0001 C CNN "Manufacturer"
+F 11 "C14663" H 7700 5350 50  0001 C CNN "LCSC"
 	1    7700 5350
 	1    0    0    -1
@@
 F 9 "" H 0   0   50  0001 C CNN "Description"
 F 10 "" H 0   0   50  0001 C CNN "Manufacturer"
+F 11 "C14663" H 7700 3550 50  0001 C CNN "LCSC"
 	1    7700 3550
 	1    0    0    -1
@@
 F 9 "" H 0   0   50  0001 C CNN "Description"
 F 10 "" H 0   0   50  0001 C CNN "Manufacturer"
+F 11 "C14663" H 5050 3550 50  0001 C CNN "LCSC"
 	1    5050 3550
 	1    0    0    -1
@@
 F 9 "" H 0   0   50  0001 C CNN "Description"
 F 10 "" H 0   0   50  0001 C CNN "Manufacturer"
+F 11 "C14663" H 5000 5350 50  0001 C CNN "LCSC"
 	1    5000 5350
 	1    0    0    -1
@@
 F 9 "" H 0   0   50  0001 C CNN "Description"
 F 10 "" H 0   0   50  0001 C CNN "Manufacturer"
+F 11 "C14663" H 2450 5350 50  0001 C CNN "LCSC"
 	1    2450 5350
 	1    0    0    -1
@@
 F 9 "" H 0   0   50  0001 C CNN "Description"
 F 10 "" H 0   0   50  0001 C CNN "Manufacturer"
+F 11 "C14663" H 6850 1500 50  0001 C CNN "LCSC"
 	1    6850 1500
 	0    -1   -1   0
@@
 F 9 "" H 0   0   50  0001 C CNN "Description"
 F 10 "" H 0   0   50  0001 C CNN "Manufacturer"
+F 11 "C14663" H 7700 2050 50  0001 C CNN "LCSC"
 	1    7700 2050
 	1    0    0    -1
@@
 F 9 "" H 0   0   50  0001 C CNN "Description"
 F 10 "" H 0   0   50  0001 C CNN "Manufacturer"
+F 11 "C14663" H 5050 2050 50  0001 C CNN "LCSC"
 	1    5050 2050
 	1    0    0    -1
