File: hw/kicad/v4.0/hv_supply.sch (KiCad schematic (older format))
At the start: 32 parts, among them U4 ACT4088, U5 LNK304D

Commit message: WIP LCSC
Parts:
- C15, C41, C58, C60: LCSC (none) -> C14663
Changed lines of the file:
@@
 EESchema Schematic File Version 4
-LIBS:stmbl_4.0-cache
-EELAYER 26 0
+EELAYER 30 0
 EELAYER END
 $Descr A4 11693 8268
@@
 F 9 "" H 0   0   50  0001 C CNN "Description"
 F 10 "" H 0   0   50  0001 C CNN "Manufacturer"
+F 11 "C14663" H 7200 4250 50  0001 C CNN "LCSC"
 	1    7200 4250
 	1    0    0    -1
@@
 F 9 "" H 0   0   50  0001 C CNN "Description"
 F 10 "" H 0   0   50  0001 C CNN "Manufacturer"
+F 11 "C14663" H 5250 3750 50  0001 C CNN "LCSC"
 	1    5250 3750
 	1    0    0    -1
@@
 F 9 "" H 0   0   50  0001 C CNN "Description"
 F 10 "" H 0   0   50  0001 C CNN "Manufacturer"
+F 11 "C14663" H 2600 5900 50  0001 C CNN "LCSC"
 	1    2600 5900
 	0    -1   -1   0
@@
 F 9 "" H 0   0   50  0001 C CNN "Description"
 F 10 "" H 0   0   50  0001 C CNN "Manufacturer"
+F 11 "C14663" H 3250 6450 50  0001 C CNN "LCSC"
 	1    3250 6450
 	1    0    0    -1
