File: hw/kicad/v4.0/io.sch (KiCad schematic (older format))
At the start: 51 parts, among them P10 CONN_02X06, P4 CONN_01X02, P5 CONN_01X06, P9 CONN_01X06, Q1 IRLML6344, Q2 IRLML6344, Q3 IRLML6344, Q4 IRLML6344

Commit message: WIP LCSC
Parts:
- C100, C130, C91, C94, C95, C98: LCSC (none) -> C14663
Changed lines of the file:
@@
 EESchema Schematic File Version 4
-LIBS:stmbl_4.0-cache
-EELAYER 26 0
+EELAYER 30 0
 EELAYER END
 $Descr A4 11693 8268
@@
 F 9 "" H 0   0   50  0001 C CNN "Description"
 F 10 "" H 0   0   50  0001 C CNN "Manufacturer"
+F 11 "C14663" H 1700 1300 50  0001 C CNN "LCSC"
 	1    1700 1300
 	1    0    0    -1
@@
 F 9 "" H 0   0   50  0001 C CNN "Description"
 F 10 "" H 0   0   50  0001 C CNN "Manufacturer"
+F 11 "C14663" H 1700 3300 50  0001 C CNN "LCSC"
 	1    1700 3300
 	1    0    0    -1
@@
 F 9 "" H 0   0   50  0001 C CNN "Description"
 F 10 "" H 0   0   50  0001 C CNN "Manufacturer"
+F 11 "C14663" H 1700 5300 50  0001 C CNN "LCSC"
 	1    1700 5300
 	1    0    0    -1
@@
 F 9 "" H 0   0   50  0001 C CNN "Description"
 F 10 "" H 0   0   50  0001 C CNN "Manufacturer"
+F 11 "C14663" H 10800 1550 50  0001 C CNN "LCSC"
 	1    10800 1550
 	1    0    0    -1
@@
 F 9 "" H 0   0   50  0001 C CNN "Description"
 F 10 "" H 0   0   50  0001 C CNN "Manufacturer"
+F 11 "C14663" H 11100 1550 50  0001 C CNN "LCSC"
 	1    11100 1550
 	1    0    0    -1
@@
 F 9 "" H 0   0   50  0001 C CNN "Description"
 F 10 "" H 0   0   50  0001 C CNN "Manufacturer"
+F 11 "C14663" H 4400 3300 50  0001 C CNN "LCSC"
 	1    4400 3300
 	1    0    0    -1
