File: hw/kicad/v4.0/io.sch (KiCad schematic (older format))
At the start: 51 parts, among them P10 CONN_02X06, P4 CONN_01X02, P5 CONN_01X06, P9 CONN_01X06, Q1 IRLML6344, Q2 IRLML6344, Q3 IRLML6344, Q4 IRLML6344

Commit message: Added LCSC # to parts in 4.3 PCB
Parts:
- C100, C130, C91, C94, C95, C98: LCSC (none) -> C14663
- C52, C59: LCSC (none) -> C1588
- D14, D15, D18, D19, D20, D4: LCSC (none) -> C2297
- D16: LCSC (none) -> C84256
- D17: LCSC (none) -> C2296
- D2, D3, D5, D7: LCSC (none) -> C86560
- Q1, Q2, Q3, Q4: LCSC (none) -> C53550
- R10, R11, R40, R9: LCSC (none) -> C23345
- R105, R108, R119, R12, R13, R14, R45, R99: LCSC (none) -> C21190
- R106, R98: LCSC (none) -> C25804
- R120, R134, R76, R83, R85: LCSC (none) -> C23179
- R20, R22, R74: LCSC (none) -> C23018
Changed lines of the file:
@@
 EESchema Schematic File Version 4
 LIBS:stmbl_4.0-cache
-EELAYER 26 0
+EELAYER 30 0
 EELAYER END
 $Descr A4 11693 8268
@@
 F 9 "" H 0   0   50  0001 C CNN "Description"
 F 10 "Infineon" H 0   0   50  0001 C CNN "Manufacturer"
+F 11 "C53550" H 2000 1850 50  0001 C CNN "LCSC"
 	1    2000 1850
 	1    0    0    -1
@@
 F 9 "" H 0   0   50  0001 C CNN "Description"
 F 10 "" H 0   0   50  0001 C CNN "Manufacturer"
+F 11 "C23345" H 1450 1900 50  0001 C CNN "LCSC"
 	1    1450 1900
 	0    1    1    0
@@
 F 9 "" H 0   0   50  0001 C CNN "Description"
 F 10 "" H 0   0   50  0001 C CNN "Manufacturer"
+F 11 "C21190" H 1700 2150 50  0001 C CNN "LCSC"
 	1    1700 2150
 	1    0    0    -1
@@
 F 9 "" H 0   0   50  0001 C CNN "Description"
 F 10 "Micro Commercial Co" H 0   0   50  0001 C CNN "Manufacturer"
+F 11 "C86560" H 2100 1300 50  0001 C CNN "LCSC"
 	1    2100 1300
 	0    1    1    0
@@
 F 9 "" H 0   0   50  0001 C CNN "Description"
 F 10 "Infineon" H 0   0   50  0001 C CNN "Manufacturer"
+F 11 "C53550" H 2000 3850 50  0001 C CNN "LCSC"
 	1    2000 3850
 	1    0    0    -1
@@
 F 9 "" H 0   0   50  0001 C CNN "Description"
 F 10 "" H 0   0   50  0001 C CNN "Manufacturer"
+F 11 "C23345" H 1450 3900 50  0001 C CNN "LCSC"
 	1    1450 3900
 	0    1    1    0
@@
 F 9 "" H 0   0   50  0001 C CNN "Description"
 F 10 "" H 0   0   50  0001 C CNN "Manufacturer"
+F 11 "C21190" H 1700 4150 50  0001 C CNN "LCSC"
 	1    1700 4150
 	1    0    0    -1
@@
 F 9 "" H 0   0   50  0001 C CNN "Description"
 F 10 "Micro Commercial Co" H 0   0   50  0001 C CNN "Manufacturer"
+F 11 "C86560" H 2100 3300 50  0001 C CNN "LCSC"
 	1    2100 3300
 	0    1    1    0
@@
 F 9 "" H 0   0   50  0001 C CNN "Description"
 F 10 "Infineon" H 0   0   50  0001 C CNN "Manufacturer"
+F 11 "C53550" H 2000 5850 50  0001 C CNN "LCSC"
 	1    2000 5850
 	1    0    0    -1
@@
 F 9 "" H 0   0   50  0001 C CNN "Description"
 F 10 "" H 0   0   50  0001 C CNN "Manufacturer"
+F 11 "C23345" H 1450 5900 50  0001 C CNN "LCSC"
 	1    1450 5900
 	0    1    1    0
@@
 F 9 "" H 0   0   50  0001 C CNN "Description"
 F 10 "" H 0   0   50  0001 C CNN "Manufacturer"
+F 11 "C21190" H 1700 6150 50  0001 C CNN "LCSC"
 	1    1700 6150
 	1    0    0    -1
@@
 F 9 "" H 0   0   50  0001 C CNN "Description"
 F 10 "Micro Commercial Co" H 0   0   50  0001 C CNN "Manufacturer"
+F 11 "C86560" H 2100 5300 50  0001 C CNN "LCSC"
 	1    2100 5300
 	0    1    1    0
@@
 F 9 "" H 0   0   50  0001 C CNN "Description"
 F 10 "Infineon" H 0   0   50  0001 C CNN "Manufacturer"
+F 11 "C53550" H 4700 3850 50  0001 C CNN "LCSC"
 	1    4700 3850
 	1    0    0    -1
@@
 F 9 "" H 0   0   50  0001 C CNN "Description"
 F 10 "" H 0   0   50  0001 C CNN "Manufacturer"
+F 11 "C23345" H 4150 3900 50  0001 C CNN "LCSC"
 	1    4150 3900
 	0    1    1    0
@@
 F 9 "" H 0   0   50  0001 C CNN "Description"
 F 10 "" H 0   0   50  0001 C CNN "Manufacturer"
+F 11 "C21190" H 4400 4150 50  0001 C CNN "LCSC"
 	1    4400 4150
 	1    0    0    -1
@@
 F 9 "" H 0   0   50  0001 C CNN "Description"
 F 10 "Micro Commercial Co" H 0   0   50  0001 C CNN "Manufacturer"
+F 11 "C86560" H 4800 3300 50  0001 C CNN "LCSC"
 	1    4800 3300
 	0    1    1    0
@@
 F 9 "" H 0   0   50  0001 C CNN "Description"
 F 10 "" H 0   0   50  0001 C CNN "Manufacturer"
+F 11 "C21190" H 10050 2350 50  0001 C CNN "LCSC"
 	1    10050 2350
 	1    0    0    -1
@@
 F 9 "" H 0   0   50  0001 C CNN "Description"
 F 10 "" H 0   0   50  0001 C CNN "Manufacturer"
+F 11 "C25804" H 9850 2350 50  0001 C CNN "LCSC"
 	1    9850 2350
 	1    0    0    -1
@@
 F 9 "" H 0   0   50  0001 C CNN "Description"
 F 10 "" H 0   0   50  0001 C CNN "Manufacturer"
+F 11 "C21190" H 9850 2850 50  0001 C CNN "LCSC"
 	1    9850 2850
 	1    0    0    -1
@@
 F 9 "" H 0   0   50  0001 C CNN "Description"
 F 10 "" H 0   0   50  0001 C CNN "Manufacturer"
+F 11 "C21190" H 9250 2350 50  0001 C CNN "LCSC"
 	1    9250 2350
 	1    0    0    -1
@@
 F 9 "" H 0   0   50  0001 C CNN "Description"
 F 10 "" H 0   0   50  0001 C CNN "Manufacturer"
+F 11 "C25804" H 9050 2350 50  0001 C CNN "LCSC"
 	1    9050 2350
 	1    0    0    -1
@@
 F 9 "" H 0   0   50  0001 C CNN "Description"
 F 10 "" H 0   0   50  0001 C CNN "Manufacturer"
+F 11 "C21190" H 9050 2850 50  0001 C CNN "LCSC"
 	1    9050 2850
 	1    0    0    -1
@@
 F 9 "" H 0   0   50  0001 C CNN "Description"
 F 10 "" H 0   0   50  0001 C CNN "Manufacturer"
+F 11 "C1588" H 9250 2850 50  0001 C CNN "LCSC"
 	1    9250 2850
 	1    0    0    -1
@@
 F 9 "" H 0   0   50  0001 C CNN "Description"
 F 10 "" H 0   0   50  0001 C CNN "Manufacturer"
+F 11 "C1588" H 10050 2850 50  0001 C CNN "LCSC"
 	1    10050 2850
 	1    0    0    -1
@@
 F 9 "" H 0   0   50  0001 C CNN "Description"
 F 10 "" H 0   0   50  0001 C CNN "Manufacturer"
+F 11 "C23018" H 2450 1400 50  0001 C CNN "LCSC"
 	1    2450 1400
 	1    0    0    -1
@@
 F 9 "" H 0   0   50  0001 C CNN "Description"
 F 10 "Lite-On" H 0   0   50  0001 C CNN "Manufacturer"
+F 11 "C2297" H 2450 1150 50  0001 C CNN "LCSC"
 	1    2450 1150
 	0    -1   -1   0
@@
 F 9 "" H 0   0   50  0001 C CNN "Description"
 F 10 "" H 0   0   50  0001 C CNN "Manufacturer"
+F 11 "C23018" H 2450 3400 50  0001 C CNN "LCSC"
 	1    2450 3400
 	1    0    0    -1
@@
 F 9 "" H 0   0   50  0001 C CNN "Description"
 F 10 "Lite-On" H 0   0   50  0001 C CNN "Manufacturer"
+F 11 "C2297" H 2450 3150 50  0001 C CNN "LCSC"
 	1    2450 3150
 	0    -1   -1   0
@@
 F 9 "" H 0   0   50  0001 C CNN "Description"
 F 10 "" H 0   0   50  0001 C CNN "Manufacturer"
+F 11 "C23018" H 2450 5400 50  0001 C CNN "LCSC"
 	1    2450 5400
 	1    0    0    -1
@@
 F 9 "" H 0   0   50  0001 C CNN "Description"
 F 10 "Lite-On" H 0   0   50  0001 C CNN "Manufacturer"
+F 11 "C2297" H 2450 5150 50  0001 C CNN "LCSC"
 	1    2450 5150
 	0    -1   -1   0
@@
 F 9 "" H 0   0   50  0001 C CNN "Description"
 F 10 "" H 0   0   50  0001 C CNN "Manufacturer"
+F 11 "C23179" H 8350 2950 50  0001 C CNN "LCSC"
 	1    8350 2950
 	1    0    0    -1
@@
 F 9 "" H 0   0   50  0001 C CNN "Description"
 F 10 "Lite-On" H 0   0   50  0001 C CNN "Manufacturer"
+F 11 "C2297" H 8350 2600 50  0001 C CNN "LCSC"
 	1    8350 2600
 	0    -1   -1   0
@@
 F 9 "" H 0   0   50  0001 C CNN "Description"
 F 10 "" H 0   0   50  0001 C CNN "Manufacturer"
+F 11 "C23179" H 7950 2950 50  0001 C CNN "LCSC"
 	1    7950 2950
 	1    0    0    -1
@@
 F 9 "" H 0   0   50  0001 C CNN "Description"
 F 10 "Lite-On" H 0   0   50  0001 C CNN "Manufacturer"
+F 11 "C2297" H 7950 2600 50  0001 C CNN "LCSC"
 	1    7950 2600
 	0    -1   -1   0
@@
 F 9 "" H 0   0   50  0001 C CNN "Description"
 F 10 "" H 0   0   50  0001 C CNN "Manufacturer"
+F 11 "C23179" H 7550 2950 50  0001 C CNN "LCSC"
 	1    7550 2950
 	1    0    0    -1
@@
 F 9 "" H 0   0   50  0001 C CNN "Description"
 F 10 "Lite-On" H 0   0   50  0001 C CNN "Manufacturer"
+F 11 "C2297" H 7550 2600 50  0001 C CNN "LCSC"
 	1    7550 2600
 	0    -1   -1   0
@@
 F 9 "" H 0   0   50  0001 C CNN "Description"
 F 10 "" H 0   0   50  0001 C CNN "Manufacturer"
+F 11 "C23179" H 7150 2950 50  0001 C CNN "LCSC"
 	1    7150 2950
 	1    0    0    -1
@@
 F 9 "" H 0   0   50  0001 C CNN "Description"
 F 10 "Lite-On" H 0   0   50  0001 C CNN "Manufacturer"
+F 11 "C2296" H 7150 2600 50  0001 C CNN "LCSC"
 	1    7150 2600
 	0    -1   -1   0
@@
 F 9 "" H 0   0   50  0001 C CNN "Description"
 F 10 "" H 0   0   50  0001 C CNN "Manufacturer"
+F 11 "C23179" H 6700 2950 50  0001 C CNN "LCSC"
 	1    6700 2950
 	1    0    0    -1
@@
 F 9 "" H 0   0   50  0001 C CNN "Description"
 F 10 "Lite-On" H 0   0   50  0001 C CNN "Manufacturer"
+F 11 "C84256" H 6700 2600 50  0001 C CNN "LCSC"
 	1    6700 2600
 	0    -1   -1   0
@@
 F 9 "" H 0   0   50  0001 C CNN "Description"
 F 10 "" H 0   0   50  0001 C CNN "Manufacturer"
+F 11 " C14663" H 1700 1300 50  0001 C CNN "LCSC"
 	1    1700 1300
 	1    0    0    -1
@@
 F 9 "" H 0   0   50  0001 C CNN "Description"
 F 10 "" H 0   0   50  0001 C CNN "Manufacturer"
+F 11 " C14663" H 1700 3300 50  0001 C CNN "LCSC"
 	1    1700 3300
 	1    0    0    -1
@@
 F 9 "" H 0   0   50  0001 C CNN "Description"
 F 10 "" H 0   0   50  0001 C CNN "Manufacturer"
+F 11 " C14663" H 1700 5300 50  0001 C CNN "LCSC"
 	1    1700 5300
 	1    0    0    -1
@@
 F 9 "" H 0   0   50  0001 C CNN "Description"
 F 10 "" H 0   0   50  0001 C CNN "Manufacturer"
+F 11 " C14663" H 10800 1550 50  0001 C CNN "LCSC"
 	1    10800 1550
 	1    0    0    -1
@@
 F 9 "" H 0   0   50  0001 C CNN "Description"
 F 10 "" H 0   0   50  0001 C CNN "Manufacturer"
+F 11 " C14663" H 11100 1550 50  0001 C CNN "LCSC"
 	1    11100 1550
 	1    0    0    -1
@@
 F 9 "" H 0   0   50  0001 C CNN "Description"
 F 10 "" H 0   0   50  0001 C CNN "Manufacturer"
+F 11 " C14663" H 4400 3300 50  0001 C CNN "LCSC"
 	1    4400 3300
 	1    0    0    -1

Commit message: Changed 120uf 1808 to 1210 100uF
Parts:
- C100, C130, C91, C94, C95, C98: LCSC C14663 -> C14663
Changed lines of the file:
@@
 F 9 "" H 0   0   50  0001 C CNN "Description"
 F 10 "" H 0   0   50  0001 C CNN "Manufacturer"
-F 11 " C14663" H 1700 1300 50  0001 C CNN "LCSC"
+F 11 "C14663" H 1700 1300 50  0001 C CNN "LCSC"
 	1    1700 1300
 	1    0    0    -1
@@
 F 9 "" H 0   0   50  0001 C CNN "Description"
 F 10 "" H 0   0   50  0001 C CNN "Manufacturer"
-F 11 " C14663" H 1700 3300 50  0001 C CNN "LCSC"
+F 11 "C14663" H 1700 3300 50  0001 C CNN "LCSC"
 	1    1700 3300
 	1    0    0    -1
@@
 F 9 "" H 0   0   50  0001 C CNN "Description"
 F 10 "" H 0   0   50  0001 C CNN "Manufacturer"
-F 11 " C14663" H 1700 5300 50  0001 C CNN "LCSC"
+F 11 "C14663" H 1700 5300 50  0001 C CNN "LCSC"
 	1    1700 5300
 	1    0    0    -1
@@
 F 9 "" H 0   0   50  0001 C CNN "Description"
 F 10 "" H 0   0   50  0001 C CNN "Manufacturer"
-F 11 " C14663" H 10800 1550 50  0001 C CNN "LCSC"
+F 11 "C14663" H 10800 1550 50  0001 C CNN "LCSC"
 	1    10800 1550
 	1    0    0    -1
@@
 F 9 "" H 0   0   50  0001 C CNN "Description"
 F 10 "" H 0   0   50  0001 C CNN "Manufacturer"
-F 11 " C14663" H 11100 1550 50  0001 C CNN "LCSC"
+F 11 "C14663" H 11100 1550 50  0001 C CNN "LCSC"
 	1    11100 1550
 	1    0    0    -1
@@
 F 9 "" H 0   0   50  0001 C CNN "Description"
 F 10 "" H 0   0   50  0001 C CNN "Manufacturer"
-F 11 " C14663" H 4400 3300 50  0001 C CNN "LCSC"
+F 11 "C14663" H 4400 3300 50  0001 C CNN "LCSC"
 	1    4400 3300
 	1    0    0    -1

Commit message: Switch some 2.2uf 0603 to 1uf bypass to get 50V version on jlcpcb
Change 2.2uf 0603 to 0805 on iram to get 50V version on jlcpcb
other cleanup
Parts:
- C100, C130, C91, C94, C95, C98: Manufacturer (none) -> YAGEO; Manufacturer No (none) -> CC0603KRX7R9BB104
- C52, C59: Manufacturer (none) -> Samsung Electro-Mechanics; Manufacturer No (none) -> CL10B102KB8NNNC
Changed lines of the file:
@@
 F 3 "" H 9250 2850 60  0000 C CNN
 F 4 "" H 9250 2850 60  0001 C CNN "InternalName"
-F 5 "" H 9250 2850 60  0001 C CNN "Manufacturer No"
+F 5 "CL10B102KB8NNNC" H 9250 2850 60  0001 C CNN "Manufacturer No"
 F 6 "50V" H 9250 2850 60  0001 C CNN "Voltage"
 F 7 "" H 9250 2850 60  0001 C CNN "Source"
 F 8 "X5R" H 9250 2850 60  0001 C CNN "Tolerance"
 F 9 "" H 0   0   50  0001 C CNN "Description"
-F 10 "" H 0   0   50  0001 C CNN "Manufacturer"
+F 10 "Samsung Electro-Mechanics" H 0   0   50  0001 C CNN "Manufacturer"
 F 11 "C1588" H 9250 2850 50  0001 C CNN "LCSC"
 	1    9250 2850
@@
 F 3 "" H 10050 2850 60  0000 C CNN
 F 4 "" H 10050 2850 60  0001 C CNN "InternalName"
-F 5 "" H 10050 2850 60  0001 C CNN "Manufacturer No"
+F 5 "CL10B102KB8NNNC" H 10050 2850 60  0001 C CNN "Manufacturer No"
 F 6 "50V" H 10050 2850 60  0001 C CNN "Voltage"
 F 7 "" H 10050 2850 60  0001 C CNN "Source"
 F 8 "X5R" H 10050 2850 60  0001 C CNN "Tolerance"
 F 9 "" H 0   0   50  0001 C CNN "Description"
-F 10 "" H 0   0   50  0001 C CNN "Manufacturer"
+F 10 "Samsung Electro-Mechanics" H 0   0   50  0001 C CNN "Manufacturer"
 F 11 "C1588" H 10050 2850 50  0001 C CNN "LCSC"
 	1    10050 2850
@@
 F 3 "" H 1700 1300 60  0000 C CNN
 F 4 "" H 1700 1300 60  0001 C CNN "InternalName"
-F 5 "" H 1700 1300 60  0001 C CNN "Manufacturer No"
+F 5 "CC0603KRX7R9BB104 " H 1700 1300 60  0001 C CNN "Manufacturer No"
 F 6 "50V" H 1700 1300 60  0001 C CNN "Voltage"
 F 7 "" H 1700 1300 60  0001 C CNN "Source"
 F 8 "X5R" H 1700 1300 60  0001 C CNN "Tolerance"
 F 9 "" H 0   0   50  0001 C CNN "Description"
-F 10 "" H 0   0   50  0001 C CNN "Manufacturer"
+F 10 "YAGEO" H 0   0   50  0001 C CNN "Manufacturer"
 F 11 "C14663" H 1700 1300 50  0001 C CNN "LCSC"
 	1    1700 1300
@@
 F 3 "" H 1700 3300 60  0000 C CNN
 F 4 "" H 1700 3300 60  0001 C CNN "InternalName"
-F 5 "" H 1700 3300 60  0001 C CNN "Manufacturer No"
+F 5 "CC0603KRX7R9BB104 " H 1700 3300 60  0001 C CNN "Manufacturer No"
 F 6 "50V" H 1700 3300 60  0001 C CNN "Voltage"
 F 7 "" H 1700 3300 60  0001 C CNN "Source"
 F 8 "X5R" H 1700 3300 60  0001 C CNN "Tolerance"
 F 9 "" H 0   0   50  0001 C CNN "Description"
-F 10 "" H 0   0   50  0001 C CNN "Manufacturer"
+F 10 "YAGEO" H 0   0   50  0001 C CNN "Manufacturer"
 F 11 "C14663" H 1700 3300 50  0001 C CNN "LCSC"
 	1    1700 3300
@@
 F 3 "" H 1700 5300 60  0000 C CNN
 F 4 "" H 1700 5300 60  0001 C CNN "InternalName"
-F 5 "" H 1700 5300 60  0001 C CNN "Manufacturer No"
+F 5 "CC0603KRX7R9BB104 " H 1700 5300 60  0001 C CNN "Manufacturer No"
 F 6 "50V" H 1700 5300 60  0001 C CNN "Voltage"
 F 7 "" H 1700 5300 60  0001 C CNN "Source"
 F 8 "X5R" H 1700 5300 60  0001 C CNN "Tolerance"
 F 9 "" H 0   0   50  0001 C CNN "Description"
-F 10 "" H 0   0   50  0001 C CNN "Manufacturer"
+F 10 "YAGEO" H 0   0   50  0001 C CNN "Manufacturer"
 F 11 "C14663" H 1700 5300 50  0001 C CNN "LCSC"
 	1    1700 5300
@@
 F 3 "" H 10800 1550 60  0000 C CNN
 F 4 "" H 10800 1550 60  0001 C CNN "InternalName"
-F 5 "" H 10800 1550 60  0001 C CNN "Manufacturer No"
+F 5 "CC0603KRX7R9BB104 " H 10800 1550 60  0001 C CNN "Manufacturer No"
 F 6 "50V" H 10800 1550 60  0001 C CNN "Voltage"
 F 7 "" H 10800 1550 60  0001 C CNN "Source"
 F 8 "X5R" H 10800 1550 60  0001 C CNN "Tolerance"
 F 9 "" H 0   0   50  0001 C CNN "Description"
-F 10 "" H 0   0   50  0001 C CNN "Manufacturer"
+F 10 "YAGEO" H 0   0   50  0001 C CNN "Manufacturer"
 F 11 "C14663" H 10800 1550 50  0001 C CNN "LCSC"
 	1    10800 1550
@@
 F 3 "" H 11100 1550 60  0000 C CNN
 F 4 "" H 11100 1550 60  0001 C CNN "InternalName"
-F 5 "" H 11100 1550 60  0001 C CNN "Manufacturer No"
+F 5 "CC0603KRX7R9BB104 " H 11100 1550 60  0001 C CNN "Manufacturer No"
 F 6 "50V" H 11100 1550 60  0001 C CNN "Voltage"
 F 7 "" H 11100 1550 60  0001 C CNN "Source"
 F 8 "X5R" H 11100 1550 60  0001 C CNN "Tolerance"
 F 9 "" H 0   0   50  0001 C CNN "Description"
-F 10 "" H 0   0   50  0001 C CNN "Manufacturer"
+F 10 "YAGEO" H 0   0   50  0001 C CNN "Manufacturer"
 F 11 "C14663" H 11100 1550 50  0001 C CNN "LCSC"
 	1    11100 1550
@@
 F 3 "" H 4400 3300 60  0000 C CNN
 F 4 "" H 4400 3300 60  0001 C CNN "InternalName"
-F 5 "" H 4400 3300 60  0001 C CNN "Manufacturer No"
+F 5 "CC0603KRX7R9BB104 " H 4400 3300 60  0001 C CNN "Manufacturer No"
 F 6 "50V" H 4400 3300 60  0001 C CNN "Voltage"
 F 7 "" H 4400 3300 60  0001 C CNN "Source"
 F 8 "X5R" H 4400 3300 60  0001 C CNN "Tolerance"
 F 9 "" H 0   0   50  0001 C CNN "Description"
-F 10 "" H 0   0   50  0001 C CNN "Manufacturer"
+F 10 "YAGEO" H 0   0   50  0001 C CNN "Manufacturer"
 F 11 "C14663" H 4400 3300 50  0001 C CNN "LCSC"
 	1    4400 3300
