File: hw/kicad/v4.0/cur.sch (KiCad schematic (older format))
At the start: 9 parts

Commit message: Added LCSC # to parts in 4.3 PCB
Parts:
- C33, C45, C57: LCSC (none) -> C1647
- R100, R46, R84: LCSC (none) -> C23179
- R107, R58, R90: LCSC (none) -> C22809
Changed lines of the file:
@@
 EESchema Schematic File Version 4
 LIBS:stmbl_4.0-cache
-EELAYER 26 0
+EELAYER 30 0
 EELAYER END
 $Descr A4 11693 8268
@@
 F 9 "" H 0   0   50  0001 C CNN "Description"
 F 10 "" H 0   0   50  0001 C CNN "Manufacturer"
+F 11 "C23179" H 4450 3000 50  0001 C CNN "LCSC"
 	1    4450 3000
 	0    1    1    0
@@
 F 9 "" H 0   0   50  0001 C CNN "Description"
 F 10 "" H 0   0   50  0001 C CNN "Manufacturer"
+F 11 "C1647" H 4700 3250 50  0001 C CNN "LCSC"
 	1    4700 3250
 	1    0    0    -1
@@
 F 9 "" H 0   0   50  0001 C CNN "Description"
 F 10 "" H 0   0   50  0001 C CNN "Manufacturer"
+F 11 "C22809" H 4700 2750 50  0001 C CNN "LCSC"
 	1    4700 2750
 	-1   0    0    1
@@
 F 9 "" H 0   0   50  0001 C CNN "Description"
 F 10 "" H 0   0   50  0001 C CNN "Manufacturer"
+F 11 "C23179" H 5650 3000 50  0001 C CNN "LCSC"
 	1    5650 3000
 	0    1    1    0
@@
 F 9 "" H 0   0   50  0001 C CNN "Description"
 F 10 "" H 0   0   50  0001 C CNN "Manufacturer"
+F 11 "C1647" H 5900 3250 50  0001 C CNN "LCSC"
 	1    5900 3250
 	1    0    0    -1
@@
 F 9 "" H 0   0   50  0001 C CNN "Description"
 F 10 "" H 0   0   50  0001 C CNN "Manufacturer"
+F 11 "C22809" H 5900 2750 50  0001 C CNN "LCSC"
 	1    5900 2750
 	-1   0    0    1
@@
 F 9 "" H 0   0   50  0001 C CNN "Description"
 F 10 "" H 0   0   50  0001 C CNN "Manufacturer"
+F 11 "C23179" H 6850 3000 50  0001 C CNN "LCSC"
 	1    6850 3000
 	0    1    1    0
@@
 F 9 "" H 0   0   50  0001 C CNN "Description"
 F 10 "" H 0   0   50  0001 C CNN "Manufacturer"
+F 11 "C1647" H 7100 3250 50  0001 C CNN "LCSC"
 	1    7100 3250
 	1    0    0    -1
@@
 F 9 "" H 0   0   50  0001 C CNN "Description"
 F 10 "" H 0   0   50  0001 C CNN "Manufacturer"
+F 11 "C22809" H 7100 2750 50  0001 C CNN "LCSC"
 	1    7100 2750
 	-1   0    0    1

Commit message: Switch some 2.2uf 0603 to 1uf bypass to get 50V version on jlcpcb
Change 2.2uf 0603 to 0805 on iram to get 50V version on jlcpcb
other cleanup
Parts:
- C33, C45, C57: Manufacturer (none) -> Samsung Electro-Mechanics; Manufacturer No (none) -> CL10C180JB8NNNC
Changed lines of the file:
@@
 F 3 "" H 4700 3250 50  0000 C CNN
 F 4 "" H 4700 3250 50  0001 C CNN "InternalName"
-F 5 "" H 4700 3250 50  0001 C CNN "Manufacturer No"
+F 5 "CL10C180JB8NNNC" H 4700 3250 50  0001 C CNN "Manufacturer No"
 F 6 "50V" H 4700 3250 50  0001 C CNN "Voltage"
 F 7 "" H 4700 3250 50  0001 C CNN "Source"
 F 8 "X5R" H 4700 3250 50  0001 C CNN "Tolerance"
 F 9 "" H 0   0   50  0001 C CNN "Description"
-F 10 "" H 0   0   50  0001 C CNN "Manufacturer"
+F 10 "Samsung Electro-Mechanics" H 0   0   50  0001 C CNN "Manufacturer"
 F 11 "C1647" H 4700 3250 50  0001 C CNN "LCSC"
 	1    4700 3250
@@
 F 3 "" H 5900 3250 50  0000 C CNN
 F 4 "" H 5900 3250 50  0001 C CNN "InternalName"
-F 5 "" H 5900 3250 50  0001 C CNN "Manufacturer No"
+F 5 "CL10C180JB8NNNC" H 5900 3250 50  0001 C CNN "Manufacturer No"
 F 6 "50V" H 5900 3250 50  0001 C CNN "Voltage"
 F 7 "" H 5900 3250 50  0001 C CNN "Source"
 F 8 "X5R" H 5900 3250 50  0001 C CNN "Tolerance"
 F 9 "" H 0   0   50  0001 C CNN "Description"
-F 10 "" H 0   0   50  0001 C CNN "Manufacturer"
+F 10 "Samsung Electro-Mechanics" H 0   0   50  0001 C CNN "Manufacturer"
 F 11 "C1647" H 5900 3250 50  0001 C CNN "LCSC"
 	1    5900 3250
@@
 F 3 "" H 7100 3250 50  0000 C CNN
 F 4 "" H 7100 3250 50  0001 C CNN "InternalName"
-F 5 "" H 7100 3250 50  0001 C CNN "Manufacturer No"
+F 5 "CL10C180JB8NNNC" H 7100 3250 50  0001 C CNN "Manufacturer No"
 F 6 "50V" H 7100 3250 50  0001 C CNN "Voltage"
 F 7 "" H 7100 3250 50  0001 C CNN "Source"
 F 8 "X5R" H 7100 3250 50  0001 C CNN "Tolerance"
 F 9 "" H 0   0   50  0001 C CNN "Description"
-F 10 "" H 0   0   50  0001 C CNN "Manufacturer"
+F 10 "Samsung Electro-Mechanics" H 0   0   50  0001 C CNN "Manufacturer"
 F 11 "C1647" H 7100 3250 50  0001 C CNN "LCSC"
 	1    7100 3250
