File: hw/kicad/v4.0/hv_sense.sch (KiCad schematic (older format))
At the start: 16 parts

Commit message: Added LCSC # to parts in 4.3 PCB
Parts:
- C11, C20, C23, C39: LCSC (none) -> C1647
- R27, R28, R32, R33, R51, R52, R77, R78: LCSC (none) -> C37158
- R29, R34, R53, R79: LCSC (none) -> C23018
Changed lines of the file:
@@
 EESchema Schematic File Version 4
 LIBS:stmbl_4.0-cache
-EELAYER 26 0
+EELAYER 30 0
 EELAYER END
 $Descr A4 11693 8268
@@
 F 9 "" H 0   0   50  0001 C CNN "Description"
 F 10 "" H 0   0   50  0001 C CNN "Manufacturer"
+F 11 "C37158" H 2900 3350 50  0001 C CNN "LCSC"
 	1    2900 3350
 	1    0    0    -1
@@
 F 9 "" H 0   0   50  0001 C CNN "Description"
 F 10 "" H 0   0   50  0001 C CNN "Manufacturer"
+F 11 "C37158" H 2900 3750 50  0001 C CNN "LCSC"
 	1    2900 3750
 	1    0    0    -1
@@
 F 9 "" H 0   0   50  0001 C CNN "Description"
 F 10 "" H 0   0   50  0001 C CNN "Manufacturer"
+F 11 "C23018" H 2900 4250 50  0001 C CNN "LCSC"
 	1    2900 4250
 	1    0    0    -1
@@
 F 9 "" H 0   0   50  0001 C CNN "Description"
 F 10 "" H 0   0   50  0001 C CNN "Manufacturer"
+F 11 "C37158" H 3700 3350 50  0001 C CNN "LCSC"
 	1    3700 3350
 	1    0    0    -1
@@
 F 9 "" H 0   0   50  0001 C CNN "Description"
 F 10 "" H 0   0   50  0001 C CNN "Manufacturer"
+F 11 "C37158" H 3700 3750 50  0001 C CNN "LCSC"
 	1    3700 3750
 	1    0    0    -1
@@
 F 9 "" H 0   0   50  0001 C CNN "Description"
 F 10 "" H 0   0   50  0001 C CNN "Manufacturer"
+F 11 "C23018" H 3700 4250 50  0001 C CNN "LCSC"
 	1    3700 4250
 	1    0    0    -1
@@
 F 9 "" H 0   0   50  0001 C CNN "Description"
 F 10 "" H 0   0   50  0001 C CNN "Manufacturer"
+F 11 "C37158" H 4500 3350 50  0001 C CNN "LCSC"
 	1    4500 3350
 	1    0    0    -1
@@
 F 9 "" H 0   0   50  0001 C CNN "Description"
 F 10 "" H 0   0   50  0001 C CNN "Manufacturer"
+F 11 "C37158" H 4500 3750 50  0001 C CNN "LCSC"
 	1    4500 3750
 	1    0    0    -1
@@
 F 9 "" H 0   0   50  0001 C CNN "Description"
 F 10 "" H 0   0   50  0001 C CNN "Manufacturer"
+F 11 "C23018" H 4500 4250 50  0001 C CNN "LCSC"
 	1    4500 4250
 	1    0    0    -1
@@
 F 9 "" H 0   0   50  0001 C CNN "Description"
 F 10 "" H 0   0   50  0001 C CNN "Manufacturer"
+F 11 "C37158" H 5400 3350 50  0001 C CNN "LCSC"
 	1    5400 3350
 	1    0    0    -1
@@
 F 9 "" H 0   0   50  0001 C CNN "Description"
 F 10 "" H 0   0   50  0001 C CNN "Manufacturer"
+F 11 "C37158" H 5400 3750 50  0001 C CNN "LCSC"
 	1    5400 3750
 	1    0    0    -1
@@
 F 9 "" H 0   0   50  0001 C CNN "Description"
 F 10 "" H 0   0   50  0001 C CNN "Manufacturer"
+F 11 "C23018" H 5400 4250 50  0001 C CNN "LCSC"
 	1    5400 4250
 	1    0    0    -1
@@
 F 9 "" H 0   0   50  0001 C CNN "Description"
 F 10 "" H 0   0   50  0001 C CNN "Manufacturer"
+F 11 "C1647" H 2700 4250 50  0001 C CNN "LCSC"
 	1    2700 4250
 	1    0    0    -1
@@
 F 9 "" H 0   0   50  0001 C CNN "Description"
 F 10 "" H 0   0   50  0001 C CNN "Manufacturer"
+F 11 "C1647" H 3500 4250 50  0001 C CNN "LCSC"
 	1    3500 4250
 	1    0    0    -1
@@
 F 9 "" H 0   0   50  0001 C CNN "Description"
 F 10 "" H 0   0   50  0001 C CNN "Manufacturer"
+F 11 "C1647" H 4300 4250 50  0001 C CNN "LCSC"
 	1    4300 4250
 	1    0    0    -1
@@
 F 9 "" H 0   0   50  0001 C CNN "Description"
 F 10 "" H 0   0   50  0001 C CNN "Manufacturer"
+F 11 "C1647" H 5200 4250 50  0001 C CNN "LCSC"
 	1    5200 4250
 	1    0    0    -1

Commit message: Switch some 2.2uf 0603 to 1uf bypass to get 50V version on jlcpcb
Change 2.2uf 0603 to 0805 on iram to get 50V version on jlcpcb
other cleanup
Parts:
- C11, C20, C23, C39: Manufacturer (none) -> Samsung Electro-Mechanics; Manufacturer No (none) -> CL10C180JB8NNNC
Changed lines of the file:
@@
 F 3 "" H 2700 4250 60  0000 C CNN
 F 4 "" H 2700 4250 60  0001 C CNN "InternalName"
-F 5 "" H 2700 4250 60  0001 C CNN "Manufacturer No"
+F 5 "CL10C180JB8NNNC" H 2700 4250 60  0001 C CNN "Manufacturer No"
 F 6 "50V" H 2700 4250 60  0001 C CNN "Voltage"
 F 7 "" H 2700 4250 60  0001 C CNN "Source"
 F 8 "X5R" H 2700 4250 60  0001 C CNN "Tolerance"
 F 9 "" H 0   0   50  0001 C CNN "Description"
-F 10 "" H 0   0   50  0001 C CNN "Manufacturer"
+F 10 "Samsung Electro-Mechanics" H 0   0   50  0001 C CNN "Manufacturer"
 F 11 "C1647" H 2700 4250 50  0001 C CNN "LCSC"
 	1    2700 4250
@@
 F 3 "" H 3500 4250 60  0000 C CNN
 F 4 "" H 3500 4250 60  0001 C CNN "InternalName"
-F 5 "" H 3500 4250 60  0001 C CNN "Manufacturer No"
+F 5 "CL10C180JB8NNNC" H 3500 4250 60  0001 C CNN "Manufacturer No"
 F 6 "50V" H 3500 4250 60  0001 C CNN "Voltage"
 F 7 "" H 3500 4250 60  0001 C CNN "Source"
 F 8 "X5R" H 3500 4250 60  0001 C CNN "Tolerance"
 F 9 "" H 0   0   50  0001 C CNN "Description"
-F 10 "" H 0   0   50  0001 C CNN "Manufacturer"
+F 10 "Samsung Electro-Mechanics" H 0   0   50  0001 C CNN "Manufacturer"
 F 11 "C1647" H 3500 4250 50  0001 C CNN "LCSC"
 	1    3500 4250
@@
 F 3 "" H 4300 4250 60  0000 C CNN
 F 4 "" H 4300 4250 60  0001 C CNN "InternalName"
-F 5 "" H 4300 4250 60  0001 C CNN "Manufacturer No"
+F 5 "CL10C180JB8NNNC" H 4300 4250 60  0001 C CNN "Manufacturer No"
 F 6 "50V" H 4300 4250 60  0001 C CNN "Voltage"
 F 7 "" H 4300 4250 60  0001 C CNN "Source"
 F 8 "X5R" H 4300 4250 60  0001 C CNN "Tolerance"
 F 9 "" H 0   0   50  0001 C CNN "Description"
-F 10 "" H 0   0   50  0001 C CNN "Manufacturer"
+F 10 "Samsung Electro-Mechanics" H 0   0   50  0001 C CNN "Manufacturer"
 F 11 "C1647" H 4300 4250 50  0001 C CNN "LCSC"
 	1    4300 4250
@@
 F 3 "" H 5200 4250 60  0000 C CNN
 F 4 "" H 5200 4250 60  0001 C CNN "InternalName"
-F 5 "" H 5200 4250 60  0001 C CNN "Manufacturer No"
+F 5 "CL10C180JB8NNNC" H 5200 4250 60  0001 C CNN "Manufacturer No"
 F 6 "50V" H 5200 4250 60  0001 C CNN "Voltage"
 F 7 "" H 5200 4250 60  0001 C CNN "Source"
 F 8 "X5R" H 5200 4250 60  0001 C CNN "Tolerance"
 F 9 "" H 0   0   50  0001 C CNN "Description"
-F 10 "" H 0   0   50  0001 C CNN "Manufacturer"
+F 10 "Samsung Electro-Mechanics" H 0   0   50  0001 C CNN "Manufacturer"
 F 11 "C1647" H 5200 4250 50  0001 C CNN "LCSC"
 	1    5200 4250
